File: Projects/Stop_light/stop_light.sch (KiCad schematic (older format))
At the start: 39 parts, among them U1 IS31LT3360, U2 IS31LT3360, U3 IS31LT3360

Commit message: just resaved
Parts:
- C1, C4, C7: symbol LED_Driver_ISSI_ALU-rescue:865080643008-SamacSys_Parts-LED_Driver_ISSI_ALU-rescue -> stop_light-rescue:865080643008-SamacSys_Parts-LED_Driver_ISSI_ALU-rescue-LED_Driver_ISSI_ALU-rescue
- C2, C3, C5, C6, C8, C9: symbol LED_Driver_ISSI_ALU-rescue:C-LED_Driver_ISSI-rescue-LED_Driver_ISSI_ALU-rescue-LED_Driver_ISSI_ALU-rescue -> stop_light-rescue:C-LED_Driver_ISSI-rescue-LED_Driver_ISSI_ALU-rescue-LED_Driver_ISSI_ALU-rescue-LED_Driver_ISSI_ALU-re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
- D1, D18, D2: symbol LED_Driver_ISSI_ALU-rescue:PMEG4010EGWX-SamacSys_Parts -> stop_light-rescue:PMEG4010EGWX-SamacSys_Parts-LED_Driver_ISSI_ALU-rescue
- L1, L2, L3: symbol LED_Driver_ISSI_ALU-rescue:INDUCTOR-LED_Driver_ISSI-rescue-LED_Driver_ISSI_ALU-rescue-LED_Driver_ISSI_ALU-rescue -> stop_light-rescue:INDUCTOR-LED_Driver_ISSI-rescue-LED_Driver_ISSI_ALU-rescue-LED_Driver_ISSI_ALU-rescue-LED_Driver_ISSI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
- R1, R2, R3, R4, R5, R8: symbol LED_Driver_ISSI_ALU-rescue:R-LED_Driver_ISSI-rescue-LED_Driver_ISSI_ALU-rescue-LED_Driver_ISSI_ALU-rescue -> stop_light-rescue:R-LED_Driver_ISSI-rescue-LED_Driver_ISSI_ALU-rescue-LED_Driver_ISSI_ALU-rescue-LED_Driver_ISSI_ALU-re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
- U1, U2, U3: symbol LED_Driver_ISSI_ALU-rescue:IS31LT3360-LED_Driver_ISSI-rescue-LED_Driver_ISSI_ALU-rescue-LED_Driver_ISSI_ALU-rescue -> stop_light-rescue:IS31LT3360-LED_Driver_ISSI-rescue-LED_Driver_ISSI_ALU-rescue-LED_Driver_ISSI_ALU-rescue-LED_Driver_IS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
Changed lines of the file:
@@
 $EndDescr
 $Comp
-L LED_Driver_ISSI_ALU-rescue:IS31LT3360-LED_Driver_ISSI-rescue-LED_Driver_ISSI_ALU-rescue-LED_Driver_ISSI_ALU-rescue U1
+L stop_light-rescue:IS31LT3360-LED_Driver_ISSI-rescue-LED_Driver_ISSI_ALU-rescue-LED_Driver_ISSI_ALU-rescue-LED_Driver_ISSI_ALU-rescue U1
 U 1 1 583A11F1
 P 6900 2300
@@
 $EndComp
 $Comp
-L LED_Driver_ISSI_ALU-rescue:INDUCTOR-LED_Driver_ISSI-rescue-LED_Driver_ISSI_ALU-rescue-LED_Driver_ISSI_ALU-rescue L1
+L stop_light-rescue:INDUCTOR-LED_Driver_ISSI-rescue-LED_Driver_ISSI_ALU-rescue-LED_Driver_ISSI_ALU-rescue-LED_Driver_ISSI_ALU-rescue L1
 U 1 1 583A1231
 P 7800 2500
@@
 $EndComp
 $Comp
-L LED_Driver_ISSI_ALU-rescue:C-LED_Driver_ISSI-rescue-LED_Driver_ISSI_ALU-rescue-LED_Driver_ISSI_ALU-rescue C3
+L stop_light-rescue:C-LED_Driver_ISSI-rescue-LED_Driver_ISSI_ALU-rescue-LED_Driver_ISSI_ALU-rescue-LED_Driver_ISSI_ALU-rescue C3
 U 1 1 583A125C
 P 8350 1950
@@
 $EndComp
 $Comp
-L LED_Driver_ISSI_ALU-rescue:C-LED_Driver_ISSI-rescue-LED_Driver_ISSI_ALU-rescue-LED_Driver_ISSI_ALU-rescue C2
+L stop_light-rescue:C-LED_Driver_ISSI-rescue-LED_Driver_ISSI_ALU-rescue-LED_Driver_ISSI_ALU-rescue-LED_Driver_ISSI_ALU-rescue C2
 U 1 1 583A1296
 P 6000 2250
@@
 $EndComp
 $Comp
-L LED_Driver_ISSI_ALU-rescue:R-LED_Driver_ISSI-rescue-LED_Driver_ISSI_ALU-rescue-LED_Driver_ISSI_ALU-rescue R1
+L stop_light-rescue:R-LED_Driver_ISSI-rescue-LED_Driver_ISSI_ALU-rescue-LED_Driver_ISSI_ALU-rescue-LED_Driver_ISSI_ALU-rescue R1
 U 1 1 583A132A
 P 6900 1350
@@
 $EndComp
 $Comp
-L LED_Driver_ISSI_ALU-rescue:GND-LED_Driver_ISSI-rescue-LED_Driver_ISSI_ALU-rescue-LED_Driver_ISSI_ALU-rescue #PWR01
+L stop_light-rescue:GND-LED_Driver_ISSI-rescue-LED_Driver_ISSI_ALU-rescue-LED_Driver_ISSI_ALU-rescue-LED_Driver_ISSI_ALU-rescue #PWR01
 U 1 1 583A1608
 P 5650 2500
@@
 $EndComp
 $Comp
-L LED_Driver_ISSI_ALU-rescue:VCC-LED_Driver_ISSI-rescue-LED_Driver_ISSI_ALU-rescue-LED_Driver_ISSI_ALU-rescue #PWR03
+L stop_light-rescue:VCC-LED_Driver_ISSI-rescue-LED_Driver_ISSI_ALU-rescue-LED_Driver_ISSI_ALU-rescue-LED_Driver_ISSI_ALU-rescue #PWR03
 U 1 1 583B1C32
 P 5650 1300
@@
 $EndComp
 $Comp
-L LED_Driver_ISSI_ALU-rescue:PMEG4010EGWX-SamacSys_Parts D1
+L stop_light-rescue:PMEG4010EGWX-SamacSys_Parts-LED_Driver_ISSI_ALU-rescue D1
 U 1 1 5C7C8997
 P 6350 1750
@@
 Connection ~ 4950 2400
 $Comp
-L LED_Driver_ISSI_ALU-rescue:R-LED_Driver_ISSI-rescue-LED_Driver_ISSI_ALU-rescue-LED_Driver_ISSI_ALU-rescue R8
+L stop_light-rescue:R-LED_Driver_ISSI-rescue-LED_Driver_ISSI_ALU-rescue-LED_Driver_ISSI_ALU-rescue-LED_Driver_ISSI_ALU-rescue R8
 U 1 1 5C85150E
 P 6250 2750
@@
 	6250 2900 5350 2900
 $Comp
-L LED_Driver_ISSI_ALU-rescue:IS31LT3360-LED_Driver_ISSI-rescue-LED_Driver_ISSI_ALU-rescue-LED_Driver_ISSI_ALU-rescue U2
+L stop_light-rescue:IS31LT3360-LED_Driver_ISSI-rescue-LED_Driver_ISSI_ALU-rescue-LED_Driver_ISSI_ALU-rescue-LED_Driver_ISSI_ALU-rescue U2
 U 1 1 5CAFF695
 P 6800 5250
@@
 $EndComp
 $Comp
-L LED_Driver_ISSI_ALU-rescue:INDUCTOR-LED_Driver_ISSI-rescue-LED_Driver_ISSI_ALU-rescue-LED_Driver_ISSI_ALU-rescue L2
+L stop_light-rescue:INDUCTOR-LED_Driver_ISSI-rescue-LED_Driver_ISSI_ALU-rescue-LED_Driver_ISSI_ALU-rescue-LED_Driver_ISSI_ALU-rescue L2
 U 1 1 5CAFF69C
 P 7700 5450
@@
 $EndComp
 $Comp
-L LED_Driver_ISSI_ALU-rescue:C-LED_Driver_ISSI-rescue-LED_Driver_ISSI_ALU-rescue-LED_Driver_ISSI_ALU-rescue C6
+L stop_light-rescue:C-LED_Driver_ISSI-rescue-LED_Driver_ISSI_ALU-rescue-LED_Driver_ISSI_ALU-rescue-LED_Driver_ISSI_ALU-rescue C6
 U 1 1 5CAFF6A4
 P 8250 4900
@@
 $EndComp
 $Comp
-L LED_Driver_ISSI_ALU-rescue:C-LED_Driver_ISSI-rescue-LED_Driver_ISSI_ALU-rescue-LED_Driver_ISSI_ALU-rescue C5
+L stop_light-rescue:C-LED_Driver_ISSI-rescue-LED_Driver_ISSI_ALU-rescue-LED_Driver_ISSI_ALU-rescue-LED_Driver_ISSI_ALU-rescue C5
 U 1 1 5CAFF6AC
 P 5900 5200
@@
 $EndComp
 $Comp
-L LED_Driver_ISSI_ALU-rescue:R-LED_Driver_ISSI-rescue-LED_Driver_ISSI_ALU-rescue-LED_Driver_ISSI_ALU-rescue R3
+L stop_light-rescue:R-LED_Driver_ISSI-rescue-LED_Driver_ISSI_ALU-rescue-LED_Driver_ISSI_ALU-rescue-LED_Driver_ISSI_ALU-rescue R3
 U 1 1 5CAFF6B3
 P 6800 4300
@@
 $EndComp
 $Comp
-L LED_Driver_ISSI_ALU-rescue:GND-LED_Driver_ISSI-rescue-LED_Driver_ISSI_ALU-rescue-LED_Driver_ISSI_ALU-rescue #PWR04
+L stop_light-rescue:GND-LED_Driver_ISSI-rescue-LED_Driver_ISSI_ALU-rescue-LED_Driver_ISSI_ALU-rescue-LED_Driver_ISSI_ALU-rescue #PWR04
 U 1 1 5CAFF6BA
 P 5550 5450
@@
 $EndComp
 $Comp
-L LED_Driver_ISSI_ALU-rescue:VCC-LED_Driver_ISSI-rescue-LED_Driver_ISSI_ALU-rescue-LED_Driver_ISSI_ALU-rescue #PWR02
+L stop_light-rescue:VCC-LED_Driver_ISSI-rescue-LED_Driver_ISSI_ALU-rescue-LED_Driver_ISSI_ALU-rescue-LED_Driver_ISSI_ALU-rescue #PWR02
 U 1 1 5CAFF6C0
 P 5550 4250
@@
 $EndComp
 $Comp
-L LED_Driver_ISSI_ALU-rescue:PMEG4010EGWX-SamacSys_Parts D2
+L stop_light-rescue:PMEG4010EGWX-SamacSys_Parts-LED_Driver_ISSI_ALU-rescue D2
 U 1 1 5CAFF74B
 P 6250 4700
@@
 Connection ~ 4850 5350
 $Comp
-L LED_Driver_ISSI_ALU-rescue:R-LED_Driver_ISSI-rescue-LED_Driver_ISSI_ALU-rescue-LED_Driver_ISSI_ALU-rescue R2
+L stop_light-rescue:R-LED_Driver_ISSI-rescue-LED_Driver_ISSI_ALU-rescue-LED_Driver_ISSI_ALU-rescue-LED_Driver_ISSI_ALU-rescue R2
 U 1 1 5CAFF75D
 P 6150 5700
@@
 $EndComp
 $Comp
-L LED_Driver_ISSI_ALU-rescue:IS31LT3360-LED_Driver_ISSI-rescue-LED_Driver_ISSI_ALU-rescue-LED_Driver_ISSI_ALU-rescue U3
+L stop_light-rescue:IS31LT3360-LED_Driver_ISSI-rescue-LED_Driver_ISSI_ALU-rescue-LED_Driver_ISSI_ALU-rescue-LED_Driver_ISSI_ALU-rescue U3
 U 1 1 5CE91534
 P 6800 8000
@@
 $EndComp
 $Comp
-L LED_Driver_ISSI_ALU-rescue:INDUCTOR-LED_Driver_ISSI-rescue-LED_Driver_ISSI_ALU-rescue-LED_Driver_ISSI_ALU-rescue L3
+L stop_light-rescue:INDUCTOR-LED_Driver_ISSI-rescue-LED_Driver_ISSI_ALU-rescue-LED_Driver_ISSI_ALU-rescue-LED_Driver_ISSI_ALU-rescue L3
 U 1 1 5CE9153A
 P 7700 8200
@@
 $EndComp
 $Comp
-L LED_Driver_ISSI_ALU-rescue:C-LED_Driver_ISSI-rescue-LED_Driver_ISSI_ALU-rescue-LED_Driver_ISSI_ALU-rescue C9
+L stop_light-rescue:C-LED_Driver_ISSI-rescue-LED_Driver_ISSI_ALU-rescue-LED_Driver_ISSI_ALU-rescue-LED_Driver_ISSI_ALU-rescue C9
 U 1 1 5CE91541
 P 8250 7650
@@
 $EndComp
 $Comp
-L LED_Driver_ISSI_ALU-rescue:C-LED_Driver_ISSI-rescue-LED_Driver_ISSI_ALU-rescue-LED_Driver_ISSI_ALU-rescue C8
+L stop_light-rescue:C-LED_Driver_ISSI-rescue-LED_Driver_ISSI_ALU-rescue-LED_Driver_ISSI_ALU-rescue-LED_Driver_ISSI_ALU-rescue C8
 U 1 1 5CE91548
 P 5900 7950
@@
 $EndComp
 $Comp
-L LED_Driver_ISSI_ALU-rescue:R-LED_Driver_ISSI-rescue-LED_Driver_ISSI_ALU-rescue-LED_Driver_ISSI_ALU-rescue R5
+L stop_light-rescue:R-LED_Driver_ISSI-rescue-LED_Driver_ISSI_ALU-rescue-LED_Driver_ISSI_ALU-rescue-LED_Driver_ISSI_ALU-rescue R5
 U 1 1 5CE9154E
 P 6800 7050
@@
 $EndComp
 $Comp
-L LED_Driver_ISSI_ALU-rescue:GND-LED_Driver_ISSI-rescue-LED_Driver_ISSI_ALU-rescue-LED_Driver_ISSI_ALU-rescue #PWR06
+L stop_light-rescue:GND-LED_Driver_ISSI-rescue-LED_Driver_ISSI_ALU-rescue-LED_Driver_ISSI_ALU-rescue-LED_Driver_ISSI_ALU-rescue #PWR06
 U 1 1 5CE91554
 P 5550 8200
@@
 $EndComp
 $Comp
-L LED_Driver_ISSI_ALU-rescue:VCC-LED_Driver_ISSI-rescue-LED_Driver_ISSI_ALU-rescue-LED_Driver_ISSI_ALU-rescue #PWR05
+L stop_light-rescue:VCC-LED_Driver_ISSI-rescue-LED_Driver_ISSI_ALU-rescue-LED_Driver_ISSI_ALU-rescue-LED_Driver_ISSI_ALU-rescue #PWR05
 U 1 1 5CE9155A
 P 5550 7000
@@
 Connection ~ 5900 7800
 $Comp
-L LED_Driver_ISSI_ALU-rescue:865080643008-SamacSys_Parts-LED_Driver_ISSI_ALU-rescue C7
+L stop_light-rescue:865080643008-SamacSys_Parts-LED_Driver_ISSI_ALU-rescue-LED_Driver_ISSI_ALU-rescue C7
 U 1 1 5CE915A8
 P 5550 7600
@@
 $EndComp
 $Comp
-L LED_Driver_ISSI_ALU-rescue:PMEG4010EGWX-SamacSys_Parts D18
+L stop_light-rescue:PMEG4010EGWX-SamacSys_Parts-LED_Driver_ISSI_ALU-rescue D18
 U 1 1 5CE915C1
 P 6250 7450
@@
 Connection ~ 4850 8100
 $Comp
-L LED_Driver_ISSI_ALU-rescue:R-LED_Driver_ISSI-rescue-LED_Driver_ISSI_ALU-rescue-LED_Driver_ISSI_ALU-rescue R4
+L stop_light-rescue:R-LED_Driver_ISSI-rescue-LED_Driver_ISSI_ALU-rescue-LED_Driver_ISSI_ALU-rescue-LED_Driver_ISSI_ALU-rescue R4
 U 1 1 5CE915D0
 P 6150 8450
@@
 	10300 7050 12050 7050
 $Comp
-L LED_Driver_ISSI_ALU-rescue:865080643008-SamacSys_Parts-LED_Driver_ISSI_ALU-rescue C4
+L stop_light-rescue:865080643008-SamacSys_Parts-LED_Driver_ISSI_ALU-rescue-LED_Driver_ISSI_ALU-rescue C4
 U 1 1 5CAFF731
 P 5550 4850
@@
 $EndComp
 $Comp
-L LED_Driver_ISSI_ALU-rescue:865080643008-SamacSys_Parts-LED_Driver_ISSI_ALU-rescue C1
+L stop_light-rescue:865080643008-SamacSys_Parts-LED_Driver_ISSI_ALU-rescue-LED_Driver_ISSI_ALU-rescue C1
 U 1 1 5C098AE6
 P 5650 1900

Commit message: added Samac libraries
Parts:
- added J1: 109159003101916, SamacSys_Parts:109159003101916, symbol SamacSys_Parts:109159003101916
Changed lines of the file:
@@
 	0    1    1    0
 $EndComp
+$Comp
+L SamacSys_Parts:109159003101916 J1
+U 1 1 5CEDE861
+P 950 4600
+F 0 "J1" H 1350 4865 50  0000 C CNN
+F 1 "109159003101916" H 1350 4774 50  0000 C CNN
+F 2 "SamacSys_Parts:109159003101916" H 1600 4700 50  0001 L CNN
+F 3 "https://componentsearchengine.com/Datasheets/1/109159003101916.pdf" H 1600 4600 50  0001 L CNN
+F 4 "Board to Board & Mezzanine Connectors 3WAY PLUG" H 1600 4500 50  0001 L CNN "Description"
+F 5 "" H 1600 4400 50  0001 L CNN "Height"
+F 6 "581-109159003101916" H 1600 4300 50  0001 L CNN "Mouser Part Number"
+F 7 "https://www.mouser.com/Search/Refine.aspx?Keyword=581-109159003101916" H 1600 4200 50  0001 L CNN "Mouser Price/Stock"
+F 8 "AVX" H 1600 4100 50  0001 L CNN "Manufacturer_Name"
+F 9 "109159003101916" H 1600 4000 50  0001 L CNN "Manufacturer_Part_Number"
+	1    950  4600
+	1    0    0    -1
+$EndComp
 $EndSCHEMATC

Commit message: updated with new connector and capacitors
Parts:
- C1, C4, C7: footprint SamacSys_Parts:CAPAE660X560N -> Capacitor_SMD:CP_Elec_6.3x5.4
- J1: symbol SamacSys_Parts:109159003101916 -> stop_light-rescue:109159003101916-SamacSys_Parts
- R5: footprint Resistors_SMD:R_1206 -> Resistor_SMD:R_1206_3216Metric
Connections:
- wire segments 105 -> 106
- no-connect marks 0 -> 2
Changed lines of the file:
@@
 Wire Wire Line
 	4950 2400 5650 2400
-Connection ~ 4950 2400
 $Comp
 L stop_light-rescue:R-LED_Driver_ISSI-rescue-LED_Driver_ISSI_ALU-rescue-LED_Driver_ISSI_ALU-rescue-LED_Driver_ISSI_ALU-rescue R8
@@
 Wire Wire Line
 	4850 5350 5550 5350
-Connection ~ 4850 5350
 $Comp
 L stop_light-rescue:R-LED_Driver_ISSI-rescue-LED_Driver_ISSI_ALU-rescue-LED_Driver_ISSI_ALU-rescue-LED_Driver_ISSI_ALU-rescue R2
@@
 Wire Wire Line
 	6150 5850 5250 5850
-Wire Wire Line
-	2300 2400 4950 2400
-Wire Wire Line
-	2200 5350 4850 5350
 Text Label 5350 2900 0    60   ~ 0
 adj
@@
 F 0 "R5" V 6880 7050 50  0000 C CNN
 F 1 "0.22" V 6800 7050 50  0000 C CNN
-F 2 "Resistors_SMD:R_1206" V 6730 7050 50  0000 C CNN
+F 2 "Resistor_SMD:R_1206_3216Metric" V 6730 7050 50  0000 C CNN
 F 3 "" H 6800 7050 50  0000 C CNN
 	1    6800 7050
@@
 F 0 "C7" V 5754 7730 50  0000 L CNN
 F 1 "22uF" V 5950 7650 50  0000 L CNN
-F 2 "SamacSys_Parts:CAPAE660X560N" H 5900 7650 50  0001 L CNN
+F 2 "Capacitor_SMD:CP_Elec_6.3x5.4" H 5900 7650 50  0001 L CNN
 F 3 "" H 5900 7550 50  0001 L CNN
 F 4 "Wurth Elektronik 22F 50 V dc Aluminium Electrolytic Capacitor, WCAP-ASLI Series 2000h 6.3 (Dia.) x 5.35mm" H 5900 7450 50  0001 L CNN "Description"
@@
 Wire Wire Line
 	4850 8100 5550 8100
-Connection ~ 4850 8100
 $Comp
 L stop_light-rescue:R-LED_Driver_ISSI-rescue-LED_Driver_ISSI_ALU-rescue-LED_Driver_ISSI_ALU-rescue-LED_Driver_ISSI_ALU-rescue R4
@@
 Wire Wire Line
 	6150 8600 5250 8600
-Wire Wire Line
-	2200 8100 4850 8100
 Text Label 5250 8600 0    60   ~ 0
 adj
@@
 F 0 "C4" V 5754 4980 50  0000 L CNN
 F 1 "22uF" V 5950 4900 50  0000 L CNN
-F 2 "SamacSys_Parts:CAPAE660X560N" H 5900 4900 50  0001 L CNN
+F 2 "Capacitor_SMD:CP_Elec_6.3x5.4" H 5900 4900 50  0001 L CNN
 F 3 "" H 5900 4800 50  0001 L CNN
 F 4 "Wurth Elektronik 22F 50 V dc Aluminium Electrolytic Capacitor, WCAP-ASLI Series 2000h 6.3 (Dia.) x 5.35mm" H 5900 4700 50  0001 L CNN "Description"
@@
 F 0 "C1" V 5854 2030 50  0000 L CNN
 F 1 "22uF" V 6050 1950 50  0000 L CNN
-F 2 "SamacSys_Parts:CAPAE660X560N" H 6000 1950 50  0001 L CNN
+F 2 "Capacitor_SMD:CP_Elec_6.3x5.4" H 6000 1950 50  0001 L CNN
 F 3 "" H 6000 1850 50  0001 L CNN
 F 4 "Wurth Elektronik 22F 50 V dc Aluminium Electrolytic Capacitor, WCAP-ASLI Series 2000h 6.3 (Dia.) x 5.35mm" H 6000 1750 50  0001 L CNN "Description"
@@
 $EndComp
 $Comp
-L SamacSys_Parts:109159003101916 J1
+L stop_light-rescue:109159003101916-SamacSys_Parts J1
 U 1 1 5CEDE861
 P 950 4600
@@
 	1    0    0    -1
 $EndComp
+NoConn ~ 950  4800
+NoConn ~ 1750 4700
+$Comp
+L stop_light-rescue:VCC-LED_Driver_ISSI-rescue-LED_Driver_ISSI_ALU-rescue-LED_Driver_ISSI_ALU-rescue-LED_Driver_ISSI_ALU-rescue #PWR0101
+U 1 1 5CF72751
+P 800 4400
+F 0 "#PWR0101" H 800 4250 50  0001 C CNN
+F 1 "VCC" H 800 4550 50  0000 C CNN
+F 2 "" H 800 4400 50  0000 C CNN
+F 3 "" H 800 4400 50  0000 C CNN
+	1    800  4400
+	1    0    0    -1
+$EndComp
+Wire Wire Line
+	800  4400 800  4600
+Wire Wire Line
+	800  4600 950  4600
+$Comp
+L stop_light-rescue:GND-LED_Driver_ISSI-rescue-LED_Driver_ISSI_ALU-rescue-LED_Driver_ISSI_ALU-rescue-LED_Driver_ISSI_ALU-rescue #PWR0102
+U 1 1 5CF769AC
+P 2150 4700
+F 0 "#PWR0102" H 2150 4450 50  0001 C CNN
+F 1 "GND" H 2150 4550 50  0000 C CNN
+F 2 "" H 2150 4700 50  0000 C CNN
+F 3 "" H 2150 4700 50  0000 C CNN
+	1    2150 4700
+	1    0    0    -1
+$EndComp
+Wire Wire Line
+	2150 4700 2150 4600
+Wire Wire Line
+	2150 4600 1750 4600
+Text Label 950  4700 2    60   ~ 0
+adj
 $EndSCHEMATC
