File: Projects/Stop_light/stop_light.kicad_pcb (KiCad board)
At the start: 2 copper layers, 148.2 x 255.8 mm, 34 parts, among them U1 IS31LT3360, U2 IS31LT3360

Commit message: added Samac libraries
Parts:
- added J1: 109159003101916, SamacSys_Parts:109159003101916, F.Cu at (587.9, 35.0)
Changed lines of the file:
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@@
     (tracks 72)
     (zones 0)
-    (modules 34)
+    (modules 35)
     (nets 26)
   )
@@
       (rotate (xyz 0 0 0))
     )
+  )
+  (module SamacSys_Parts:109159003101916 (layer F.Cu)
+    (at 587.94 34.97)
+    (descr 109159003101916)
+    (tags Connector)
+    (attr smd)
+    (fp_text reference J1 (at -3.916 0.897) (layer F.SilkS)
+      (effects (font (size 1.27 1.27) (thickness 0.254)))
+    )
+    (fp_text value 109159003101916 (at -3.916 0.897) (layer F.SilkS) hide
+      (effects (font (size 1.27 1.27) (thickness 0.254)))
+    )
+    (fp_text user %R (at -3.916 0.897) (layer F.Fab)
+      (effects (font (size 1.27 1.27) (thickness 0.254)))
+    )
+    (fp_line (start -5.5 -2.2) (end 5.5 -2.2) (layer F.Fab) (width 0.2))
+    (fp_line (start 5.5 -2.2) (end 5.5 0.3) (layer F.Fab) (width 0.2))
+    (fp_line (start 5.5 0.3) (end -5.5 0.3) (layer F.Fab) (width 0.2))
+    (fp_line (start -5.5 0.3) (end -5.5 -2.2) (layer F.Fab) (width 0.2))
+    (fp_line (start -5.5 -2.2) (end 5.5 -2.2) (layer F.SilkS) (width 0.2))
+    (fp_line (start -5.5 0.3) (end -4 0.3) (layer F.SilkS) (width 0.2))
+    (fp_line (start 5.5 0.3) (end 4 0.3) (layer F.SilkS) (width 0.2))
+    (pad 1 smd rect (at 3 0) (size 1.2 2) (layers F.Cu F.Paste))
+    (pad 2 smd rect (at 0 0) (size 1.2 2) (layers F.Cu F.Paste))
+    (pad 3 smd rect (at -3 0) (size 1.2 2) (layers F.Cu F.Paste))
+    (pad 4 smd rect (at -5.5 -0.95) (size 1.5 1.6) (layers F.Cu F.Paste))
+    (pad 5 smd rect (at 5.5 -0.95) (size 1.5 1.6) (layers F.Cu F.Paste))
   )
   (gr_line (start 535.627277 84.54239) (end 531.41341 74.493501) (layer Edge.Cuts) (width 0.2))
@@
   (segment (start 591.97 94.865) (end 591.025 94.865) (width 1) (layer F.Cu) (net 3) (status 10))
   (segment (start 591.025 94.865) (end 590.2862 94.865) (width 1) (layer F.Cu) (net 3) (status 20))
-  (segment (start 576.86 123.04) (end 576.86 123.79) (width 0.5) (layer F.Cu) (net 3))
-  (segment (start 576.86 123.79) (end 576.86 124.59) (width 0.5) (layer F.Cu) (net 3))
+  (segment (start 576.86 123.04) (end 576.86 123.79) (width 0.5) (layer F.Cu) (net 3) (status 30))
+  (segment (start 576.86 123.79) (end 576.86 124.59) (width 0.5) (layer F.Cu) (net 3) (status 30))
   (segment (start 576.86 125.39) (end 577.87 126.4) (width 0.5) (layer F.Cu) (net 3))
-  (segment (start 576.86 124.59) (end 576.86 125.39) (width 0.5) (layer F.Cu) (net 3))
+  (segment (start 576.86 124.59) (end 576.86 125.39) (width 0.5) (layer F.Cu) (net 3) (status 10))
   (segment (start 577.87 126.4) (end 581.76 126.4) (width 0.5) (layer F.Cu) (net 3))
-  (segment (start 581.76 102.6468) (end 589.914 94.4928) (width 0.5) (layer F.Cu) (net 3))
+  (segment (start 581.76 102.6468) (end 589.914 94.4928) (width 0.5) (layer F.Cu) (net 3) (status 20))
   (segment (start 581.76 126.4) (end 581.76 102.6468) (width 0.5) (layer F.Cu) (net 3))
   (segment (start 589.914 90.9678) (end 589.914 91.6928) (width 1) (layer F.Cu) (net 4) (status 20))
@@
   (segment (start 596.778 89.751) (end 595.51199 88.48499) (width 1) (layer F.Cu) (net 4))
   (segment (start 600.328 89.751) (end 596.778 89.751) (width 1) (layer F.Cu) (net 4) (status 10))
-  (segment (start 549.11 59.435) (end 549.11 58.87) (width 0.5) (layer F.Cu) (net 4))
+  (segment (start 549.11 59.435) (end 549.11 58.87) (width 0.5) (layer F.Cu) (net 4) (status 30))
   (segment (start 549.11 58.07) (end 549.31 57.87) (width 0.5) (layer F.Cu) (net 4))
-  (segment (start 549.11 58.87) (end 549.11 58.07) (width 0.5) (layer F.Cu) (net 4))
+  (segment (start 549.11 58.87) (end 549.11 58.07) (width 0.5) (layer F.Cu) (net 4) (status 10))
   (segment (start 549.31 57.87) (end 556.93 57.87) (width 0.5) (layer F.Cu) (net 4))
   (segment (start 556.93 58.7088) (end 567.9 69.6788) (width 0.5) (layer F.Cu) (net 4))
   (segment (start 556.93 57.87) (end 556.93 58.7088) (width 0.5) (layer F.Cu) (net 4))
   (segment (start 567.9 69.6788) (end 567.9 78.29) (width 0.5) (layer F.Cu) (net 4))
-  (segment (start 581.3028 91.6928) (end 589.914 91.6928) (width 0.5) (layer F.Cu) (net 4))
+  (segment (start 581.3028 91.6928) (end 589.914 91.6928) (width 0.5) (layer F.Cu) (net 4) (status 20))
   (segment (start 567.9 78.29) (end 581.3028 91.6928) (width 0.5) (layer F.Cu) (net 4))
   (segment (start 601.12 94.693) (end 600.328 93.901) (width 1) (layer F.Cu) (net 5) (status 30))
@@
   (segment (start 596.617 91.565) (end 598.953 93.901) (width 1) (layer F.Cu) (net 5) (status 20))
   (segment (start 594.97 91.565) (end 596.617 91.565) (width 1) (layer F.Cu) (net 5) (status 10))
-  (segment (start 569.4 107.58) (end 569.4 108.33) (width 0.5) (layer F.Cu) (net 6))
-  (segment (start 569.4 108.33) (end 569.4 109.13) (width 0.5) (layer F.Cu) (net 6))
-  (segment (start 569.4 113.39) (end 569.4 109.13) (width 0.5) (layer F.Cu) (net 6))
-  (segment (start 576.86 121.65) (end 576.86 120.85) (width 0.5) (layer F.Cu) (net 6))
+  (segment (start 569.4 107.58) (end 569.4 108.33) (width 0.5) (layer F.Cu) (net 6) (status 30))
+  (segment (start 569.4 108.33) (end 569.4 109.13) (width 0.5) (layer F.Cu) (net 6) (status 30))
+  (segment (start 569.4 113.39) (end 569.4 109.13) (width 0.5) (layer F.Cu) (net 6) (status 20))
+  (segment (start 576.86 121.65) (end 576.86 120.85) (width 0.5) (layer F.Cu) (net 6) (status 10))
   (segment (start 576.86 120.85) (end 569.4 113.39) (width 0.5) (layer F.Cu) (net 6))
-  (segment (start 569.4 106.755) (end 569.4 106.19) (width 0.5) (layer F.Cu) (net 7))
-  (segment (start 562.31 94.02) (end 562.31 93.5) (width 0.5) (layer F.Cu) (net 7))
+  (segment (start 569.4 106.755) (end 569.4 106.19) (width 0.5) (layer F.Cu) (net 7) (status 30))
+  (segment (start 562.31 94.02) (end 562.31 93.5) (width 0.5) (layer F.Cu) (net 7) (status 20))
   (segment (start 562.31 98.3) (end 562.31 94.02) (width 0.5) (layer F.Cu) (net 7))
-  (segment (start 569.4 106.19) (end 569.4 105.39) (width 0.5) (layer F.Cu) (net 7))
+  (segment (start 569.4 106.19) (end 569.4 105.39) (width 0.5) (layer F.Cu) (net 7) (status 10))
   (segment (start 569.4 105.39) (end 562.31 98.3) (width 0.5) (layer F.Cu) (net 7))
   (segment (start 562.31 91.125) (end 562.31 90.56) (width 0.5) (layer F.Cu) (net 8) (status 30))
-  (segment (start 555.55 83) (end 555.55 77.71) (width 0.5) (layer F.Cu) (net 8))
-  (segment (start 562.31 90.56) (end 562.31 89.76) (width 0.5) (layer F.Cu) (net 8))
+  (segment (start 555.55 83) (end 555.55 77.71) (width 0.5) (layer F.Cu) (net 8) (status 20))
+  (segment (start 562.31 90.56) (end 562.31 89.76) (width 0.5) (layer F.Cu) (net 8) (status 10))
   (segment (start 562.31 89.76) (end 555.55 83) (width 0.5) (layer F.Cu) (net 8))
-  (segment (start 549.11 67.53) (end 549.11 61.81) (width 0.5) (layer F.Cu) (net 9))
-  (segment (start 555.55 74.77) (end 555.55 73.97) (width 0.5) (layer F.Cu) (net 9))
+  (segment (start 549.11 67.53) (end 549.11 61.81) (width 0.5) (layer F.Cu) (net 9) (status 20))
+  (segment (start 555.55 74.77) (end 555.55 73.97) (width 0.5) (layer F.Cu) (net 9) (status 10))
   (segment (start 555.55 73.97) (end 549.11 67.53) (width 0.5) (layer F.Cu) (net 9))
-  (segment (start 549.11 61.81) (end 549.11 61.01) (width 0.5) (layer F.Cu) (net 9))
-  (segment (start 549.11 61.01) (end 549.11 60.26) (width 0.5) (layer F.Cu) (net 9))
+  (segment (start 549.11 61.81) (end 549.11 61.01) (width 0.5) (layer F.Cu) (net 9) (status 30))
+  (segment (start 549.11 61.01) (end 549.11 60.26) (width 0.5) (layer F.Cu) (net 9) (status 30))
   (segment (start 591.97 90.56) (end 591.97 91.565) (width 0.5) (layer F.Cu) (net 20) (status 20))
   (segment (start 592.72 89.81) (end 591.97 90.56) (width 0.5) (layer F.Cu) (net 20) (status 10))

Commit message: minor edits to kicad_pcb file
Parts:
- added C7: 22uF, SamacSys_Parts:CAPAE660X560N, F.Cu at (546.1, -63.0)
- added D18: PMEG4010EGWX, SamacSys_Parts:SOD3616X130N, F.Cu at (543.7, -57.4)
- added L3: 47uH, SRN6045TA-6R8M:SRN6045, F.Cu at (554.1, -63.6)
- added U3: IS31LT3360, Kicad_mylib:SOT89-5_JOOL, F.Cu at (553.4, -58.1)
Connections:
- R4 pad 1: (no net) -> Net-(R4-Pad1)
Changed lines of the file:
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@@
-(kicad_pcb (version 20171130) (host pcbnew "(5.1.2)-1")
+(kicad_pcb (version 20171130) (host pcbnew "(5.0.2)-1")
   (general
     (thickness 1.6)
@@
     (tracks 72)
     (zones 0)
-    (modules 35)
-    (nets 26)
+    (modules 39)
+    (nets 28)
   )
   (page A4)
@@
     (zone_45_only no)
     (trace_min 0.2)
+    (segment_width 0.2)
+    (edge_width 0.15)
     (via_size 0.6)
     (via_drill 0.4)
@@
     (uvia_min_size 0.2)
     (uvia_min_drill 0.1)
-    (edge_width 0.15)
-    (segment_width 0.2)
     (pcb_text_width 0.3)
     (pcb_text_size 1.5 1.5)
@@
   (net 24 "Net-(C9-Pad1)")
   (net 25 "Net-(C9-Pad2)")
+  (net 26 "Net-(D18-Pad2)")
+  (net 27 "Net-(R4-Pad1)")
   (net_class Default "This is the default net class."
     (clearance 0.2)
@@
     (add_net "Net-(D15-Pad1)")
     (add_net "Net-(D16-Pad1)")
+    (add_net "Net-(D18-Pad2)")
     (add_net "Net-(D2-Pad2)")
     (add_net "Net-(D3-Pad1)")
@@
     (add_net "Net-(D8-Pad1)")
     (add_net "Net-(R2-Pad1)")
+    (add_net "Net-(R4-Pad1)")
     (add_net "Net-(R8-Pad1)")
   )
@@
       (effects (font (size 0.8 0.8) (thickness 0.12)))
     )
-    (pad 1 smd roundrect (at -1.4 0) (size 1.25 1.75) (layers F.Cu F.Paste F.Mask) (roundrect_rratio 0.2))
+    (pad 1 smd roundrect (at -1.4 0) (size 1.25 1.75) (layers F.Cu F.Paste F.Mask) (roundrect_rratio 0.2)
+      (net 27 "Net-(R4-Pad1)"))
     (pad 2 smd roundrect (at 1.4 0) (size 1.25 1.75) (layers F.Cu F.Paste F.Mask) (roundrect_rratio 0.2)
       (net 22 /adj))
@@
     (pad 5 smd rect (at 5.5 -0.95) (size 1.5 1.6) (layers F.Cu F.Paste))
   )
+  (module SamacSys_Parts:CAPAE660X560N (layer F.Cu)
+    (at 546.050001 -62.974999)
+    (descr WCAP)
+    (tags "Capacitor Polarised")
+    (attr smd)
+    (fp_text reference C7 (at 0 0) (layer F.SilkS)
+      (effects (font (size 1.27 1.27) (thickness 0.254)))
+    )
+    (fp_text value 22uF (at 0 0) (layer F.SilkS) hide
+      (effects (font (size 1.27 1.27) (thickness 0.254)))
+    )
+    (fp_line (start -4.925 -3.9) (end 4.925 -3.9) (layer Dwgs.User) (width 0.05))
+    (fp_line (start 4.925 -3.9) (end 4.925 3.9) (layer Dwgs.User) (width 0.05))
+    (fp_line (start 4.925 3.9) (end -4.925 3.9) (layer Dwgs.User) (width 0.05))
+    (fp_line (start -4.925 3.9) (end -4.925 -3.9) (layer Dwgs.User) (width 0.05))
+    (fp_line (start 3.3 -3.3) (end -1.65 -3.3) (layer Dwgs.User) (width 0.1))
+    (fp_line (start -1.65 -3.3) (end -3.3 -1.65) (layer Dwgs.User) (width 0.1))
+    (fp_line (start -3.3 -1.65) (end -3.3 1.65) (layer Dwgs.User) (width 0.1))
+    (fp_line (start -3.3 1.65) (end -1.65 3.3) (layer Dwgs.User) (width 0.1))
+    (fp_line (start -1.65 3.3) (end 3.3 3.3) (layer Dwgs.User) (width 0.1))
+    (fp_line (start 3.3 3.3) (end 3.3 -3.3) (layer Dwgs.User) (width 0.1))
+    (fp_line (start -4.425 -3.3) (end 3.3 -3.3) (layer F.SilkS) (width 0.2))
+    (fp_line (start -1.65 3.3) (end 3.3 3.3) (layer F.SilkS) (width 0.2))
+    (pad 1 smd rect (at -2.75 0 90) (size 1.8 3.35) (layers F.Cu F.Paste F.Mask)
+      (net 1 VCC))
+    (pad 2 smd rect (at 2.75 0 90) (size 1.8 3.35) (layers F.Cu F.Paste F.Mask)
+      (net 2 GND))
+  )
+  (module SamacSys_Parts:SOD3616X130N (layer F.Cu)
+    (at 543.650001 -57.374999)
+    (descr SOD123_1)
+    (tags "Schottky Diode")
+    (attr smd)
+    (fp_text reference D18 (at 0 0) (layer F.SilkS)
+      (effects (font (size 1.27 1.27) (thickness 0.254)))
+    )
+    (fp_text value PMEG4010EGWX (at 0 0) (layer F.SilkS) hide
+      (effects (font (size 1.27 1.27) (thickness 0.254)))
+    )
+    (fp_line (start -2.525 -1.65) (end 2.525 -1.65) (layer Dwgs.User) (width 0.05))
+    (fp_line (start 2.525 -1.65) (end 2.525 1.65) (layer Dwgs.User) (width 0.05))
+    (fp_line (start 2.525 1.65) (end -2.525 1.65) (layer Dwgs.User) (width 0.05))
+    (fp_line (start -2.525 1.65) (end -2.525 -1.65) (layer Dwgs.User) (width 0.05))
+    (fp_line (start -1.338 -0.8) (end 1.338 -0.8) (layer Dwgs.User) (width 0.1))
+    (fp_line (start 1.338 -0.8) (end 1.338 0.8) (layer Dwgs.User) (width 0.1))
+    (fp_line (start 1.338 0.8) (end -1.338 0.8) (layer Dwgs.User) (width 0.1))
+    (fp_line (start -1.338 0.8) (end -1.338 -0.8) (layer Dwgs.User) (width 0.1))
+    (fp_line (start -1.338 -0.175) (end -0.712 -0.8) (layer Dwgs.User) (width 0.1))
+    (fp_line (start -2.275 -0.8) (end 1.338 -0.8) (layer F.SilkS) (width 0.2))
+    (fp_line (start -1.338 0.8) (end 1.338 0.8) (layer F.SilkS) (width 0.2))
+    (pad 1 smd rect (at -1.65 0 90) (size 0.8 1.25) (layers F.Cu F.Paste F.Mask)
+      (net 1 VCC))
+    (pad 2 smd rect (at 1.65 0 90) (size 0.8 1.25) (layers F.Cu F.Paste F.Mask)
+      (net 26 "Net-(D18-Pad2)"))
+  )
+  (module SRN6045TA-6R8M:SRN6045 (layer F.Cu)
+    (at 554.062501 -63.65)
+    (attr smd)
+    (fp_text reference L3 (at -0.5 -4) (layer F.SilkS)
+      (effects (font (size 0.787402 0.787402) (thickness 0.05)))
+    )
+    (fp_text value 47uH (at 0 0) (layer F.SilkS)
+      (effects (font (size 1 0.9) (thickness 0.05)))
+    )
+    (fp_line (start -2 3) (end 2 3) (layer F.SilkS) (width 0.125))
+    (fp_line (start 2 3) (end 3 2) (layer F.SilkS) (width 0.125))
+    (fp_line (start 3 2) (end 3 -2) (layer F.SilkS) (width 0.125))
+    (fp_line (start 3 -2) (end 2 -3) (layer F.SilkS) (width 0.125))
+    (fp_line (start 2 -3) (end -2 -3) (layer F.SilkS) (width 0.125))
+    (fp_line (start -2 -3) (end -3 -2) (layer F.SilkS) (width 0.125))
+    (fp_line (start -3 -2) (end -3 2) (layer F.SilkS) (width 0.125))
+    (fp_line (start -3 2) (end -2 3) (layer F.SilkS) (width 0.125))
+    (pad 1 smd rect (at 0 -2.075) (size 5.1 2.35) (layers F.Cu F.Paste F.Mask)
+      (net 26 "Net-(D18-Pad2)"))
+    (pad 2 smd rect (at 0 2.075) (size 5.1 2.35) (layers F.Cu F.Paste F.Mask)
+      (net 25 "Net-(C9-Pad2)"))
+  )
+  (module Kicad_mylib:SOT89-5_JOOL (layer F.Cu)
+    (at 553.350001 -58.145)
+    (descr SOT89-5)
+    (tags "Integrated Circuit")
+    (attr smd)
+    (fp_text reference U3 (at -0.416 -2.538) (layer F.SilkS)
+      (effects (font (size 1.27 1.27) (thickness 0.254)))
+    )
+    (fp_text value IS31LT3360 (at -0.416 -2.538) (layer F.SilkS) hide
+      (effects (font (size 1.27 1.27) (thickness 0.254)))
+    )
+    (fp_line (start -2.25 -1.25) (end 2.25 -1.25) (layer Dwgs.User) (width 0.2))
+    (fp_line (start 2.25 -1.25) (end 2.25 1.25) (layer Dwgs.User) (width 0.2))
+    (fp_line (start 2.25 1.25) (end -2.25 1.25) (layer Dwgs.User) (width 0.2))
+    (fp_line (start -2.25 1.25) (end -2.25 -1.25) (layer Dwgs.User) (width 0.2))
+    (fp_line (start -2.25 1.25) (end -2.25 -1.25) (layer F.SilkS) (width 0.2))
+    (fp_line (start 2.25 -1.25) (end 2.25 1.25) (layer F.SilkS) (width 0.2))
+    (fp_circle (center -1.532 2.628) (end -1.549 2.628) (layer F.SilkS) (width 0.254))
+    (pad 1 smd rect (at -1.5 1.65) (size 0.68 1.2) (layers F.Cu F.Paste F.Mask)
+      (net 26 "Net-(D18-Pad2)"))
+    (pad 2 smd rect (at 0 1.55) (size 0.68 1.4) (layers F.Cu F.Paste F.Mask)
+      (net 2 GND))
+    (pad 3 smd rect (at 1.5 1.65) (size 0.68 1.2) (layers F.Cu F.Paste F.Mask)
+      (net 27 "Net-(R4-Pad1)"))
+    (pad 4 smd rect (at 1.5 -1.65) (size 0.68 1.2) (layers F.Cu F.Paste F.Mask)
+      (net 24 "Net-(C9-Pad1)"))
+    (pad 5 smd rect (at -1.5 -1.65) (size 0.68 1.2) (layers F.Cu F.Paste F.Mask)
+      (net 1 VCC))
+    (pad 2 smd rect (at 0 -0.605) (size 1.5 3.3) (layers F.Cu F.Paste F.Mask)
+      (net 2 GND))
+  )
   (gr_line (start 535.627277 84.54239) (end 531.41341 74.493501) (layer Edge.Cuts) (width 0.2))

Commit message: updated with new connector and capacitors
Parts:
- added R5: 0.22, Resistor_SMD:R_1206_3216Metric, F.Cu at (560.7, -23.5)
- C1, C4, C7: footprint SamacSys_Parts:CAPAE660X560N -> Capacitor_SMD:CP_Elec_6.3x5.4
- moved R2 93.5 mm to (566.3, -6.43), turned to 90 degrees
- moved D1 71.9 mm to (583.9, 27.7)
- moved U1 71.9 mm to (576.3, 23.4)
- moved R1 71.9 mm to (576.3, 27.2)
- moved R8 71.9 mm to (575.5, 18.6)
- moved C1 71.9 mm to (578.3, 33.4)
- moved C2 71.9 mm to (580.1, 27.6)
- moved C3 71.9 mm to (572.7, 23.3)
- moved L1 71.9 mm to (583.1, 22.0)
- moved R4 51.2 mm to (559.7, -32.1), turned to 90 degrees
- moved C7 48.3 mm to (562.3, -17.5), turned to 270 degrees
- moved C9 44.1 mm to (557.1, -27.3), turned to 90 degrees
- moved D18 41.0 mm to (567.6, -24.1), turned to 90 degrees
- moved L3 35.8 mm to (566.9, -30.2), turned to 180 degrees
- moved C4 32.6 mm to (569.0, 8.27), turned to 270 degrees
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Connections:
- J1 pad 1: (no net) -> VCC
- J1 pad 2: (no net) -> GND
- J1 pad 3: (no net) -> /adj
Routing:
- net Net-(C9-Pad2): track 0.00 -> 131.3 mm
- net /adj: track 0.00 -> 75.3 mm
- net Net-(C3-Pad1): track 48.1 -> 119.4 mm
- net Net-(C6-Pad1): track 0.00 -> 70.2 mm
- net Net-(C6-Pad2): track 0.00 -> 65.1 mm
- net Net-(C9-Pad1): track 0.00 -> 49.7 mm
- net GND: track 20.5 -> 46.5 mm
- net Net-(D8-Pad1): track 0.00 -> 15.6 mm
- net Net-(D10-Pad1): track 0.00 -> 15.6 mm
- net Net-(D10-Pad2): track 0.00 -> 15.6 mm
- net Net-(D11-Pad1): track 0.00 -> 15.6 mm
- net Net-(D13-Pad1): track 0.00 -> 15.5 mm
- net Net-(D14-Pad1): track 0.00 -> 15.5 mm
- net Net-(D15-Pad1): track 0.00 -> 15.5 mm
- net Net-(D16-Pad1): track 0.00 -> 15.4 mm
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
Commit message: stop light updated
Parts:
- D3, D4, D5: footprint myKicad_lib:DMLQ31_23 -> myKicad_lib:DMLQ31_23_Large_pad
- R1: value 0.22 -> 0.3; footprint Resistors_SMD:R_1206 -> Resistor_SMD:R_1206_3216Metric
- R3, R5: value 0.22 -> 0.3
- moved J1 10.6 mm to (593.2, 49.4), turned to 286.4 degrees
- moved C7 9.96 mm to (556.8, -25.8)
- moved C8 9.96 mm to (559.0, -31.5)
- moved C9 9.96 mm to (551.6, -35.6)
- moved D18 9.96 mm to (562.1, -32.4)
- moved R5 9.96 mm to (555.2, -31.8)
- moved L3 9.96 mm to (561.4, -38.5)
- moved R4 9.96 mm to (554.2, -40.4)
- moved U3 9.96 mm to (555.2, -35.6)
- moved C5 9.60 mm to (566.5, -5.90)
- moved C6 9.57 mm to (559.3, -10.2)
- moved L2 9.57 mm to (569.5, -11.6)
- moved C4 9.57 mm to (564.6, -0.23)
- moved D2 9.57 mm to (570.4, -5.83)
- moved R2 9.57 mm to (561.9, -14.9)
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Connections:
- J1 pad 1: VCC -> /adj
- J1 pad 3: /adj -> VCC
Routing:
- net /adj: track 75.3 -> 585.2 mm
- net GND: track 46.5 -> 168.5 mm
- net VCC: track 29.3 -> 140.0 mm
- net Net-(C9-Pad2): track 131.3 -> 119.5 mm
- net Net-(C6-Pad2): track 65.1 -> 57.2 mm
- net Net-(C6-Pad1): track 70.2 -> 77.6 mm
- net Net-(C9-Pad1): track 49.7 -> 45.4 mm
- net Net-(C3-Pad1): track 119.4 -> 123.5 mm
- net Net-(C3-Pad2): track 66.2 -> 67.2 mm
- net Net-(D3-Pad1): track 17.2 -> 17.7 mm
- net Net-(D8-Pad1): track 15.6 -> 16.2 mm
Other:
- outline, holes or cut-outs redrawn
- net class VCC: clearance 0.2 -> 0.3; trace_width 1 -> 0.7
- net class power: clearance 0.2 -> 0.3; trace_width 1 -> 0.7

Commit message: added fabrication files for stop light
Parts:
- added REF**: mountinghole4mm, myKicad_lib:mountinghole4mm, F.Cu at (523.8, -98.3)
- added REF**: mountinghole4mm, myKicad_lib:mountinghole4mm, F.Cu at (539.0, -33.2)
- added REF**: mountinghole4mm, myKicad_lib:mountinghole4mm, F.Cu at (559.0, 26.7)
- added REF**: mountinghole4mm, myKicad_lib:mountinghole4mm, F.Cu at (596.4, 121.6)
- added REF**: mountinghole4mm, myKicad_lib:mountinghole4mm, F.Cu at (578.9, 76.8)
- D10, D11, D12, D13, D14, D15, D16, D17, D6, D7, D8, D9: footprint myKicad_lib:DMLQ31_23 -> myKicad_lib:DMLQ31_23_Large_pad
- D3: footprint myKicad_lib:DMLQ31_23_Large_pad -> myKicad_lib:DMLQ31_23_Large_pad_solder_paste
Routing:
- net Net-(D10-Pad2): track 15.6 -> 17.7 mm
- net Net-(D10-Pad1): track 15.6 -> 17.7 mm
- net Net-(D11-Pad1): track 15.6 -> 17.7 mm
- net Net-(D15-Pad1): track 15.5 -> 17.6 mm
- net Net-(D14-Pad1): track 15.5 -> 17.6 mm
- net Net-(D13-Pad1): track 15.5 -> 17.6 mm
- net Net-(D16-Pad1): track 15.4 -> 17.5 mm
- net Net-(D8-Pad1): track 16.2 -> 17.7 mm
- net Net-(D5-Pad1): track 16.2 -> 17.8 mm
- net Net-(C9-Pad1): track 45.4 -> 47.0 mm
- net Net-(C6-Pad2): track 57.2 -> 58.6 mm
- net Net-(C9-Pad2): track 119.5 -> 120.1 mm
- net Net-(D6-Pad1): track 17.2 -> 17.7 mm
