File: Projects/Control_board/Control_board.sch (KiCad schematic (older format))
At the start: 48 parts, among them IC1 BD1HD500FVM-CTR, J1 505567-0681, J2 43045-0200, J3 43045-0200, J4 43045-0200, J5 43045-0401, J6 Conn_01x06, J8 Conn_01x02, K3 PB114024, Q1 BSS138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

Commit message: added LED with fan project
Parts:
- removed J1: 505567-0681, SamacSys_Parts:5055670681, symbol Connector_Generic:Conn_01x08
- removed J5: 43045-0401, SamacSys_Parts:430450401, symbol Control_board-rescue:43045-0401-SamacSys_Parts-Control_board-rescue-Control_boa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
- added J1: 505567-0871, 5055670871, symbol SamacSys_Parts:505567-0871
- added J5: 43045-0401, SamacSys_Parts:430450401, symbol SamacSys_Parts:43045-0401
Connections:
- wire segments 165 -> 166
Changed lines of the file:
@@
 NoConn ~ 10650 5400
-$Comp
-L Control_board-rescue:43045-0401-SamacSys_Parts-Control_board-rescue-Control_board-rescue J5
-U 1 1 5C75F026
-P 9100 7500
-F 0 "J5" V 9454 7628 50  0000 L CNN
-F 1 "43045-0401" V 9545 7628 50  0000 L CNN
-F 2 "SamacSys_Parts:430450401" H 9750 7600 50  0001 L CNN
-F 3 "http://www.mouser.com/datasheet/2/276/0430450401_PCB_HEADERS-142810.pdf" H 9750 7500 50  0001 L CNN
-F 4 "Molex MICRO-FIT 3.0 Series, Series Number 43045, 3mm Pitch 4 Way 2 Row Right Angle PCB Header, Solder Termination, 5A" H 9750 7400 50  0001 L CNN "Description"
-F 5 "8" H 9750 7300 50  0001 L CNN "Height"
-F 6 "538-43045-0401" H 9750 7200 50  0001 L CNN "Mouser Part Number"
-F 7 "Molex" H 9750 7100 50  0001 L CNN "Manufacturer_Name"
-F 8 "43045-0401" H 9750 7000 50  0001 L CNN "Manufacturer_Part_Number"
-	1    9100 7500
-	1    0    0    -1
-$EndComp
 $Comp
 L power:GND #PWR0135
@@
 Wire Wire Line
 	7900 1250 7900 3150
-Text Label 11750 2350 0    50   ~ 0
-NTC
 $Comp
 L power:+36V #PWR015
 U 1 1 5C8C2FA1
-P 12100 1800
-F 0 "#PWR015" H 12100 1650 50  0001 C CNN
-F 1 "+36V" H 12115 1973 50  0000 C CNN
-F 2 "" H 12100 1800 50  0001 C CNN
-F 3 "" H 12100 1800 50  0001 C CNN
-	1    12100 1800
-	1    0    0    -1
-$EndComp
-$Comp
-L power:GND #PWR017
-U 1 1 5C8C3004
-P 12250 2150
-F 0 "#PWR017" H 12250 1900 50  0001 C CNN
-F 1 "GND" H 12255 1977 50  0000 C CNN
-F 2 "" H 12250 2150 50  0001 C CNN
-F 3 "" H 12250 2150 50  0001 C CNN
-	1    12250 2150
-	1    0    0    -1
-$EndComp
-Text Label 11750 2550 0    50   ~ 0
-12V_Fan
-Wire Wire Line
-	12250 2150 11750 2150
-Wire Wire Line
-	11750 2250 12100 2250
-Wire Wire Line
-	12100 1800 12100 2250
+P 11800 1400
+F 0 "#PWR015" H 11800 1250 50  0001 C CNN
+F 1 "+36V" H 11815 1573 50  0000 C CNN
+F 2 "" H 11800 1400 50  0001 C CNN
+F 3 "" H 11800 1400 50  0001 C CNN
+	1    11800 1400
+	1    0    0    -1
+$EndComp
 $Comp
 L Sensor_Optical:LDR03 R4
@@
 Wire Wire Line
 	14350 5250 14250 5250
-$Comp
-L Connector_Generic:Conn_01x08 J1
-U 1 1 5CA02812
-P 11550 2450
-F 0 "J1" H 11470 1825 50  0000 C CNN
-F 1 "505567-0681" H 11470 1916 50  0000 C CNN
-F 2 "SamacSys_Parts:5055670681" H 11550 2450 50  0001 C CNN
-F 3 "~" H 11550 2450 50  0001 C CNN
-	1    11550 2450
-	-1   0    0    1
-$EndComp
 $Comp
 L Control_board-rescue:BSP76_E6433-SamacSys_Parts Q5
@@
 Text Label 7650 3350 0    50   ~ 0
 ADJ
-Text Label 11750 2050 0    50   ~ 0
+Text Label 11400 1600 0    50   ~ 0
 ADJ_LED
 Text Label 13650 8400 0    50   ~ 0
@@
 Text Label 13650 8200 0    50   ~ 0
 LDR
+$Comp
+L SamacSys_Parts:43045-0401 J5
+U 1 1 5CFE9C0C
+P 9100 7500
+F 0 "J5" H 9500 7765 50  0000 C CNN
+F 1 "43045-0401" H 9500 7674 50  0000 C CNN
+F 2 "SamacSys_Parts:430450401" H 9750 7600 50  0001 L CNN
+F 3 "http://www.mouser.com/datasheet/2/276/0430450401_PCB_HEADERS-142810.pdf" H 9750 7500 50  0001 L CNN
+F 4 "Molex MICRO-FIT 3.0 Series, Series Number 43045, 3mm Pitch 4 Way 2 Row Right Angle PCB Header, Solder Termination, 5A" H 9750 7400 50  0001 L CNN "Description"
+F 5 "8" H 9750 7300 50  0001 L CNN "Height"
+F 6 "538-43045-0401" H 9750 7200 50  0001 L CNN "Mouser Part Number"
+F 7 "Molex" H 9750 7100 50  0001 L CNN "Manufacturer_Name"
+F 8 "43045-0401" H 9750 7000 50  0001 L CNN "Manufacturer_Part_Number"
+	1    9100 7500
+	1    0    0    -1
+$EndComp
+$Comp
+L SamacSys_Parts:505567-0871 J1
+U 1 1 5CFCA1AA
+P 10500 1300
+F 0 "J1" H 10950 1565 50  0000 C CNN
+F 1 "505567-0871" H 10950 1474 50  0000 C CNN
+F 2 "5055670871" H 11250 1400 50  0001 L CNN
+F 3 "https://componentsearchengine.com/Datasheets/1/505567-0871.pdf" H 11250 1300 50  0001 L CNN
+F 4 "Headers & Wire Housings MicroLockPlus 1.25MM RA HDR SR 8CKT BLK" H 11250 1200 50  0001 L CNN "Description"
+F 5 "4" H 11250 1100 50  0001 L CNN "Height"
+F 6 "538-505567-0871" H 11250 1000 50  0001 L CNN "Mouser Part Number"
+F 7 "https://www.mouser.com/Search/Refine.aspx?Keyword=538-505567-0871" H 11250 900 50  0001 L CNN "Mouser Price/Stock"
+F 8 "Molex" H 11250 800 50  0001 L CNN "Manufacturer_Name"
+F 9 "505567-0871" H 11250 700 50  0001 L CNN "Manufacturer_Part_Number"
+	1    10500 1300
+	1    0    0    -1
+$EndComp
+Wire Wire Line
+	11800 1400 11800 1500
+Wire Wire Line
+	11800 1500 11400 1500
+$Comp
+L power:GND #PWR?
+U 1 1 5CFD25A9
+P 10150 1650
+F 0 "#PWR?" H 10150 1400 50  0001 C CNN
+F 1 "GND" H 10155 1477 50  0000 C CNN
+F 2 "" H 10150 1650 50  0001 C CNN
+F 3 "" H 10150 1650 50  0001 C CNN
+	1    10150 1650
+	1    0    0    -1
+$EndComp
+Wire Wire Line
+	10150 1650 10150 1600
+Wire Wire Line
+	10150 1600 10500 1600
+Text Label 10500 1400 2    50   ~ 0
+12V_Fan
+Text Label 10500 1500 2    50   ~ 0
+NTC
 $EndSCHEMATC

Commit message: added pca96...
Parts:
- removed J1: 505567-0871, 5055670871, symbol SamacSys_Parts:505567-0871
- removed J6: Conn_01x06, Connector_PinHeader_2.54mm:PinHeader_1x06_P2.54mm_Vertical, symbol Connector_Generic:Conn_01x06
- removed SW1, SW2: SW_Push, SamacSys_Parts:B3U-1000P, symbol Switch:SW_Push
- removed U1: ESP8266-12E_ESP-12E, ESP8266-12E_ESP-12E:XCVR_ESP8266-12E%2fESP-12E, symbol Control_board-rescue:ESP8266-12E_ESP-12E-ESP8266-12E_ESP-12E-Control_board-resc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
- removed U3: LM1117-3.3, SamacSys_Parts:SOT230P700X180-4N, symbol Regulator_Linear:LM1117-3.3
- added C5: 1uF, Capacitor_SMD:C_0603_1608Metric, symbol Device:C_Small
- added IC2: PCA9615DPJ, SamacSys_Parts:QFN50P300X300X100-10N-D, symbol SamacSys_Parts:PCA9615DPJ
- added J1: 5055780871, footprints:5055780871, symbol My_symbol_library:5055780871
- added J6: RJ45, Connector_RJ:RJ45_Amphenol_54602-x08_Horizontal, symbol Connector:RJ45
- added R15: 10K, Resistor_SMD:R_0603_1608Metric, symbol Device:R
- added R16, R18: 390, Resistor_SMD:R_0603_1608Metric, symbol Device:R
- added R17: 100, Resistor_SMD:R_0603_1608Metric, symbol Device:R
- C4: value 1uF -> 0.1uF
- R10, R3: value 10k -> 390
- R9: value 10k -> 100
Connections:
- net +36V: now also J1.4
- net +3V3: now also C4.1, R5.1, R7.1, IC2.1 (VDD(A)), J1.8, J6.4; no longer C4.2, R10.1, R3.1, R9.1
- net +5V: now also R3.1, C5.2, IC2.10 (VDD(B)), R16.1; no longer R5.1, R7.1
- net 12V_Fan: now also J1.7
- net ADJ_LED: now also J1.2
- net GND: now also C4.2, R10.2, C5.1, IC2.5 (VSS), J1.3, J6.5, R15.2, R18.2; no longer C4.1
- net NTC: now also J1.5, R15.1
- net mistmaker: now also A1.25 (A6); no longer A1.5 (D2)
- net pump: now also A1.26 (A7); no longer A1.9 (D6)
- net at A1.23 (A4), R5.2, U2.5 (SDA): now also IC2.2 (SDA)
- net at A1.24 (A5), R7.2, U2.6 (SCL): now also IC2.4 (SCL)
- net DSDA-: now reaches R9.2
- net DSDA-: now also R10.1, IC2.9 (DSDAM), J6.7
- net DSDA+: now reaches R3.2
- net DSDA+: now also R9.1, IC2.8 (DSDAP), J6.8
- new net DSCL+: IC2.7 (DSCLP), J6.2, R16.2, R17.1
- new net DSCL-: IC2.6 (DSCLM), J6.1, R17.2, R18.1
- new net EN: A1.5 (D2), IC2.3 (EN)
- no-connect marks 4 -> 10
Other:
- note added: "Buzzer"
- moved on the sheet: BT1, C1, J5, Q1, R1, R2, U2, Y1

Commit message: updates to Control board and LED light
Connections:
- net fan_+12V is gone; now on net 12V_Fan: IC1.3 (OUT_1), IC1.4 (OUT_2)
- net +3V3: now also C1.1, U2.8 (VCC)
- net heating_element: no longer names the net of A1.7 (D4)
- no-connect marks 10 -> 24
Changed lines of the file:
@@
 EESchema Schematic File Version 4
 LIBS:Control_board-cache
-EELAYER 26 0
+EELAYER 29 0
 EELAYER END
 $Descr A3 16535 11693
@@
 Text Label 5200 10050 0    50   ~ 0
 mistmaker
-Text Label 6650 2450 2    50   ~ 0
+Text Label 6400 2450 2    50   ~ 0
 airstone_pump
-Text Label 6650 2550 2    50   ~ 0
+Text Label 6400 2550 2    50   ~ 0
 fan
-Text Label 7650 3650 0    50   ~ 0
+Text Label 7750 3650 0    50   ~ 0
 mistmaker
 $Comp
@@
 Text Label 7000 8750 2    50   ~ 0
 Temp_data_3V3
-Text Label 6650 2750 2    50   ~ 0
+Text Label 6400 2750 2    50   ~ 0
 Temp_data_3V3
 $Comp
@@
 Text Label 4050 3900 0    50   ~ 0
 pump
-Text Label 6650 2850 2    50   ~ 0
-heating_element
 $Comp
 L power:+36V #PWR05
@@
 	4100 7850 4000 7850
 NoConn ~ 2800 7650
-Text Label 4000 7750 0    50   ~ 0
-fan_+12V
 Text Label 2800 7550 2    50   ~ 0
 fan_status
-Text Label 6650 2950 2    50   ~ 0
+Text Label 6400 2950 2    50   ~ 0
 fan_status
 $Comp
@@
 Wire Wire Line
 	5550 10050 5200 10050
-Text Label 7650 3750 0    50   ~ 0
+Text Label 7750 3750 0    50   ~ 0
 pump
 Text Label 7650 3350 0    50   ~ 0
@@
 Text Label 10800 7000 2    50   ~ 0
 EN
-Text Label 6650 2650 2    50   ~ 0
+Text Label 6400 2650 2    50   ~ 0
 EN
 $Comp
@@
 Wire Wire Line
 	10600 7200 10800 7200
+Text Label 4100 7750 0    50   ~ 0
+12V_Fan
+Wire Wire Line
+	6400 2450 6650 2450
+Wire Wire Line
+	6400 2550 6650 2550
+Wire Wire Line
+	6400 2650 6650 2650
+Wire Wire Line
+	6400 2750 6650 2750
+Wire Wire Line
+	6400 2950 6650 2950
+Wire Wire Line
+	7650 3650 7750 3650
+Wire Wire Line
+	7650 3750 7750 3750
+NoConn ~ 6650 2850
+NoConn ~ 6650 3050
+NoConn ~ 6650 3150
+NoConn ~ 6650 3250
+NoConn ~ 6650 3350
+NoConn ~ 6650 3450
+NoConn ~ 6650 3550
+NoConn ~ 6650 3650
+NoConn ~ 7050 2050
+NoConn ~ 7350 2050
+NoConn ~ 7650 2450
+NoConn ~ 7650 2550
+NoConn ~ 7650 2850
+NoConn ~ 7650 3050
+$Comp
+L power:PWR_FLAG #FLG0101
+U 1 1 5D5E9D88
+P 13600 7800
+F 0 "#FLG0101" H 13600 7875 50  0001 C CNN
+F 1 "PWR_FLAG" H 13600 7973 50  0000 C CNN
+F 2 "" H 13600 7800 50  0001 C CNN
+F 3 "~" H 13600 7800 50  0001 C CNN
+	1    13600 7800
+	1    0    0    -1
+$EndComp
+Wire Wire Line
+	13600 7800 13600 7900
+Wire Wire Line
+	13600 7900 14100 7900
+Connection ~ 14100 7900
+$Comp
+L power:+3.3V #PWR0131
+U 1 1 5D5F4327
+P 11350 4450
+F 0 "#PWR0131" H 11350 4300 50  0001 C CNN
+F 1 "+3.3V" H 11365 4623 50  0000 C CNN
+F 2 "" H 11350 4450 50  0001 C CNN
+F 3 "" H 11350 4450 50  0001 C CNN
+	1    11350 4450
+	1    0    0    -1
+$EndComp
+Wire Wire Line
+	11350 4450 11350 4550
+Connection ~ 11350 4550
 $EndSCHEMATC
