File: Projects/Control_board/Control_board.sch (KiCad schematic (older format))
At the start: 76 parts, among them IC1 VN7050ASTR, IC2 PCA9615DPJ, IC3 PSSI2021SAY,115, J1 66200621022, J10 43045-0401, J11 Conn_01x04, J12 Conn_01x04, J13 Conn_01x01_Female, J2 66200621022, J3 43045-0200, J4 43045-0200, J5 43045-0401, J6 RJ45, J7 66200621022, J8 Conn_01x02, Q1 Q_NMOS_GSD, Q2 BSS138-Transistor_FET, Q3 BSP76_E6433, Q5 BSP76_E6433, U1 ESP32-DEVKITC-32D, U2 NCP1117-5.0_SOT223, U4 DCDC_lm2596

Commit message: updated with reverse polarity protection
Parts:
- removed C1, C2, C6: 100nF, Capacitor_SMD:C_0603_1608Metric, symbol Control_board-rescue:C-Device
- removed D4, D5, D6, D7, D8, D9: SMF5.0A, Diode_SMD:D_SOD-123F, symbol Control_board-rescue:1.5KExxA-Diode
- removed D?: BZX84C8V2L, symbol Device:D_Zener
- removed D?: BAT54S, Package_TO_SOT_SMD:SOT-23, symbol Diode:BAT54S
- removed R?: 100, Resistor_SMD:R_0603_1608Metric, symbol Control_board-rescue:R-Device
- removed U2: NCP1117-5.0_SOT223, Package_TO_SOT_SMD:SOT-223-3_TabPin2, symbol Control_board-rescue:NCP1117-5.0_SOT223-Regulator_Linear
- removed U4: DCDC_lm2596, Kicad_mylib:LM2596_module, symbol Control_board-rescue:DCDC_lm2596-my_library2-Control_board-rescue-Control_board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
- added C1, C2, C6: 0.1uF, Capacitor_SMD:C_0603_1608Metric, symbol Control_board-rescue:C_Small-Device
- added D4, D5, D6, D7, D8, D9: BAT54S, Package_TO_SOT_SMD:SOT-23, symbol Diode:BAT54S
- added R26, R27, R30: 1k, Resistor_SMD:R_0603_1608Metric, symbol Control_board-rescue:R-Device
- added R28, R29: 10K, Resistor_SMD:R_0603_1608Metric, symbol Control_board-rescue:R-Device
- added R32, R33, R34, R35: DNP, Resistor_SMD:R_0603_1608Metric, symbol Control_board-rescue:R-Device
- added S1, S2: FSM8JRT, SamacSys_Parts:FSM8JRT, symbol SamacSys_Parts:FSM8JRT
- added U3: NID35-12_meanwell, Converter_DCDC:Converter_DCDC_MeanWell_NID30_THT, symbol my_library:NID35-12_meanwell
- added Z11: BZX84C8V2LT1G, SamacSys_Parts:SOT95P237X111-3N, symbol SamacSys_Parts:D_Zener_ALT_PELLE
- F1: renamed from F?; footprint (none) -> Fuse:Fuse_Bourns_MF-RHT1100; Manufacturer_Part_Number (none) -> 0ZRP0400FF1A
- R14, R20, R8: value 100 -> 1k
- R31: renamed from R?; footprint (none) -> Resistor_SMD:R_0603_1608Metric
- gave numbers to parts that had none: 3
Connections:
- net +12V: now also U2.3 (VI), U3.1 (Vout+), U3.2 (Vout+), U3.3 (Vout+), U3.4 (Vout+)
- net +3V3: now also D4.2, D5.2, D6.2, D7.2, D8.2, D9.2, R28.1, R29.1, R32.1
- net +48V: now also U3.7 (+Vin), U3.8 (+Vin), Z11.3 (K); no longer J8.1 (Pin_1)
- net +5V: now also U2.2 (VO)
- net GND: now also U2.1 (GND), C1.2, C2.2, C6.2, D4.1, D5.1, D6.1, D7.1, D8.1, D9.1, R33.2, S1.1, S2.2, U3.5 (COM), U3.6 (COM), Z11.1 (A)
- net NTC_1: now also R30.1; no longer R19.1, U1.27 (IO19)
- net NTC_2: now also R27.2; no longer R15.1, U1.8 (IO33)
- net NTC_3: now also R26.2; no longer R13.1, U1.7 (IO32)
- net VCC: now also J8.1 (Pin_1)
- net at J5.3, Q1.2 (S), R22.2: now also R35.2; no longer J10.3
- net Spare: now reaches U1.12 (IO14)
- net Spare: now also R32.2, R33.1, R34.1
- net at U1.25 (IO21): now also R29.2, S2.1
- net at R8.2, U1.28 (IO18): now also C1.1, D6.3
- net at R14.2, U1.34 (IO2): now also C2.1, D7.3
- net at R20.2, U1.35 (IO15): now also C6.1, D8.3
- net at U1.6 (IO35): now also R28.2, S1.2
- new net: D5.3, R15.1, R27.1, U1.8 (IO33)
- new net: D9.3, R19.1, R30.2, U1.27 (IO19)
- new net: D4.3, R13.1, R26.1, U1.7 (IO32)
- new net: J10.3, R34.2, R35.1
- no-connect marks 22 -> 23
Other:
- note removed: "3.3V IO\nPWM source (1 kHz)"
- note removed: "To light module, this pin could potentially get +48V DC"
- moved on the sheet: C7, D1, D10, D2, D3, F1, IC1, J3, J4, J8, LS1, Q2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

Commit message: updated PCB
Parts:
- removed J1: 66200621022, SamacSys_Parts:66200621022, symbol Control_board-rescue:66200621022-SamacSys_Parts
- removed J10, J5: 43045-0401, SamacSys_Parts:430450401, symbol Control_board-rescue:43045-0401-SamacSys_Parts
- removed J8: Conn_01x02, Connector_Wire:SolderWirePad_1x02_P7.62mm_Drill2mm, symbol Control_board-rescue:Conn_01x02-Connector_Generic
- removed R4: LDR03, LED_SMD:LED_0805_2012Metric, symbol Control_board-rescue:LDR03-Sensor_Optical
- added D11: BAT54W, Package_TO_SOT_SMD:SOT-323_SC-70, symbol Diode:BAT54W
- added J1: 66200621022, SamacSys_Parts:66200621022, symbol SamacSys_Parts:66200621022_0
- added J10, J5: 43045-0401_2, SamacSys_Parts:430450401, symbol SamacSys_Parts:43045-0401_2
- added J8: TB003-500-P02BE, SamacSys_Parts:SHDR2W100P0X500_1X2_1000X780X1030P, symbol SamacSys_Parts:TB003-500-P02BE
- added Q6: Q_Photo_NPN, Diode_SMD:D_1210_3225Metric_Pad1.42x2.65mm_HandSolder, symbol Device:Q_Photo_NPN
- added R4: DNP, Resistor_SMD:R_0603_1608Metric, symbol Control_board-rescue:R-Device
- D10: Manufacturer_Part_Number (none) -> SMF60A; Mouser Part Number (none) -> 576-SMF60A
- D4, D5, D6, D7, D8, D9: value BAT54S -> BAT54SLT1G; footprint Package_TO_SOT_SMD:SOT-23 -> SamacSys_Parts:SOT96P237X111-3N; Description (none) -> RLBAT54SLT1G ON Semiconductor BAT54SLT1G Rectifier Diode, 0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; Height (none) -> 1.11; Manufacturer_Name (none) -> ON Semiconductor; Manufacturer_Part_Number (none) -> BAT54SLT1G; Mouser Part Number (none) -> 863-BAT54SLT1G; Mouser Price/Stock (none) -> https://www.mouser.com/Search/Refine.aspx?Keyword=863-BAT54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
- J6: Manufacturer_Part_Number (none) -> 54602-908LF
- Q2: Manufacturer_Part_Number (none) -> BSS138A-TP
- U1: Field4 ESP32-DEVKITC-32D -> (none); Manufacturer_Part_Number (none) -> ESP32-DEVKITC-32D
- U2: Manufacturer_Part_Number (none) -> NCP1117DT50G; Mouser Part Number (none) -> 863-NCP1117DT50G
- U3: Manufacturer_Part_Number (none) -> NID35-12; Mouser Part Number (none) -> 709-NID35-12
Connections:
- net +12V: now also R4.1
- net +3V3: now also R6.1, D11.3 (K), J1.6, J10.1, J5.1; no longer U1.1 (3V3)
- net +48V: now also J1.4
- net 12V_Fan: now also J1.5
- net ADJ_LED1: now also J1.2
- net GND: now also J1.1, J10.3, J5.3, J8.2, Q6.2 (E); no longer R6.2
- net NTC_1: now also J1.3
- net VCC: now also J8.1
- net at C7.1, R21.1: now also R6.2, Q6.1 (C); no longer R6.1
- net at Q1.2 (S), R22.2, R35.2: now also J5.2
- net at R34.2, R35.1: now also J10.2
- new net: D11.1 (A), U1.1 (3V3)
- new net: J10.4, R4.2
- no-connect marks 23 -> 22
Other:
- note added: "36 Euro BOM cost"
- note added: "This mosfet is obsolete\n"
- moved on the sheet: H1, H2, H3, H4, IC3, Q1, R22, R24, R25, R32, R33, R34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
