File: Projects/Control_board/_autosave-Control_board.sch (KiCad schematic (older format))
At the start: 76 parts, among them IC1 VN7050ASTR, IC2 PCA9615DPJ, IC3 PSSI2021SAY,115, J1 66200621022, J10 43045-0401, J11 Conn_01x04, J12 Conn_01x04, J13 Conn_01x01_Female, J2 66200621022, J3 43045-0200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

Commit message: added code
Parts:
- added RV?: R_POT, symbol Device:R_POT
- added SW? (x2): SW_Push, symbol Switch:SW_Push
Changed lines of the file:
@@
 Wire Wire Line
 	9050 -600 9850 -600
+$Comp
+L Device:R_POT RV?
+U 1 1 5E6F370B
+P 3950 -1150
+F 0 "RV?" H 3881 -1104 50  0000 R CNN
+F 1 "R_POT" H 3881 -1195 50  0000 R CNN
+F 2 "" H 3950 -1150 50  0001 C CNN
+F 3 "~" H 3950 -1150 50  0001 C CNN
+	1    3950 -1150
+	1    0    0    -1
+$EndComp
+$Comp
+L Switch:SW_Push SW?
+U 1 1 5E6F5168
+P 3100 -1100
+F 0 "SW?" H 3100 -815 50  0000 C CNN
+F 1 "SW_Push" H 3100 -906 50  0000 C CNN
+F 2 "" H 3100 -900 50  0001 C CNN
+F 3 "~" H 3100 -900 50  0001 C CNN
+	1    3100 -1100
+	1    0    0    -1
+$EndComp
+$Comp
+L Switch:SW_Push SW?
+U 1 1 5E6F550C
+P 2450 -1100
+F 0 "SW?" H 2450 -815 50  0000 C CNN
+F 1 "SW_Push" H 2450 -906 50  0000 C CNN
+F 2 "" H 2450 -900 50  0001 C CNN
+F 3 "~" H 2450 -900 50  0001 C CNN
+	1    2450 -1100
+	1    0    0    -1
+$EndComp
 $EndSCHEMATC
