File: Projects/LED_DRIVER_with_fan/LED_Driver_ISSI_ALU.sch (KiCad schematic (older format))
At the start: 23 parts, among them J1 5055780871, J2 505578-0271, U1 IS31LT3360

Commit message: added pca96...
Parts:
- removed R2: LDR03, OptoDevice:R_LDR_10x8.5mm_P7.6mm_Vertical, symbol Sensor_Optical:LDR03
Connections:
- net labels added: 12V_Fan, 3.3V, 36V+, NTC
- wire segments 74 -> 69
- no-connect marks 4 -> 6
Other:
- moved on the sheet: J1
Changed lines of the file:
@@
-	1    0    0    -1
-$EndComp
-$Comp
-L Sensor_Optical:LDR03 R2
-U 1 1 5C7C2402
-P 1500 4950
-F 0 "R2" H 1570 4996 50  0000 L CNN
-F 1 "LDR03" H 1570 4905 50  0000 L CNN
-F 2 "OptoDevice:R_LDR_10x8.5mm_P7.6mm_Vertical" V 1675 4950 50  0001 C CNN
-F 3 "http://www.elektronica-componenten.nl/WebRoot/StoreNL/Shops/61422969/54F1/BA0C/C664/31B9/2173/C0A8/2AB9/2AEF/LDR03IMP.pdf" H 1500 4900 50  0001 C CNN
-	1    1500 4950
-	1    0    0    -1
-$EndComp
-$Comp
-L power:GND #PWR0101
-U 1 1 5C7C2768
-P 1500 5300
-F 0 "#PWR0101" H 1500 5050 50  0001 C CNN
-F 1 "GND" H 1505 5127 50  0000 C CNN
-F 2 "" H 1500 5300 50  0001 C CNN
-F 3 "" H 1500 5300 50  0001 C CNN
-	1    1500 5300
 	1    0    0    -1
 $EndComp
 Wire Wire Line
-	2050 5100 2050 5150
-Wire Wire Line
-	2050 5150 1500 5150
-Wire Wire Line
-	1500 5150 1500 5100
-Wire Wire Line
-	1500 5150 1500 5300
-Connection ~ 1500 5150
-Wire Wire Line
 	2050 4800 2050 2950
-Wire Wire Line
-	1500 3050 1500 4800
 Wire Wire Line
 	2700 2850 2700 2100
@@
 Wire Wire Line
 	1250 2950 2050 2950
-Wire Wire Line
-	1250 3050 1500 3050
 NoConn ~ 1250 3350
 $Comp
@@
 L LED_Driver_ISSI_ALU-rescue:5055780871 J1
 U 1 1 5C7DD705
-P 450 2800
-F 0 "J1" H 906 3437 60  0000 C CNN
-F 1 "5055780871" H 906 3331 60  0000 C CNN
-F 2 "Kicad_mylib:5055780871" H 450 2800 60  0001 C CNN
-F 3 "" H 450 2800 60  0001 C CNN
-	1    450  2800
+P 600 2850
+F 0 "J1" H 1056 3487 60  0000 C CNN
+F 1 "5055780871" H 1056 3381 60  0000 C CNN
+F 2 "Kicad_mylib:5055780871" H 600 2850 60  0001 C CNN
+F 3 "" H 600 2850 60  0001 C CNN
+	1    600  2850
 	1    0    0    -1
 $EndComp
@@
 Wire Wire Line
 	3750 3450 3750 3750
-Wire Wire Line
-	3750 3750 2150 3750
-Wire Wire Line
-	2150 3750 2150 3250
-Wire Wire Line
-	2150 3250 1250 3250
 NoConn ~ 2550 3550
 NoConn ~ 3550 3550
@@
 Wire Wire Line
 	2700 1700 2700 1250
+NoConn ~ 1250 2450
+Text Label 1250 3150 0    60   ~ 0
+12V_Fan
+Text Label 1250 2950 0    60   ~ 0
+NTC
+Text Label 1250 2850 0    60   ~ 0
+36V+
+Text Label 1250 2750 0    60   ~ 0
+GND
+$Comp
+L LED_Driver_ISSI_ALU-rescue:GND-LED_Driver_ISSI-rescue-LED_Driver_ISSI_ALU-rescue-LED_Driver_ISSI_ALU-rescue #PWR0101
+U 1 1 5D1A3668
+P 3750 3750
+F 0 "#PWR0101" H 3750 3500 50  0001 C CNN
+F 1 "GND" H 3750 3600 50  0000 C CNN
+F 2 "" H 3750 3750 50  0000 C CNN
+F 3 "" H 3750 3750 50  0000 C CNN
+	1    3750 3750
+	1    0    0    -1
+$EndComp
+Wire Wire Line
+	2050 5100 2050 5350
+Wire Wire Line
+	1500 3250 1250 3250
+Wire Wire Line
+	1500 5350 2050 5350
+Wire Wire Line
+	1500 3250 1500 5350
+Text Label 1250 3250 0    60   ~ 0
+3.3V
+NoConn ~ 1250 3050
 $EndSCHEMATC

Commit message: updates to Control board and LED light
Parts:
- J2: symbol SamacSys_Parts:505578-0271 -> LED_Driver_ISSI_ALU-rescue:505578-0271-SamacSys_Parts
Changed lines of the file:
@@
 EESchema Schematic File Version 4
 LIBS:LED_Driver_ISSI_ALU-cache
-EELAYER 26 0
+EELAYER 29 0
 EELAYER END
 $Descr A3 16535 11693
@@
 $EndComp
 $Comp
-L SamacSys_Parts:505578-0271 J2
+L LED_Driver_ISSI_ALU-rescue:505578-0271-SamacSys_Parts J2
 U 1 1 5C7DDF94
 P 2550 3450
