File: Projects/LED_DRIVER_with_fan/LED_Driver_ISSI_ALU.kicad_pcb (KiCad board)
At the start: 2 copper layers, 117.7 x 117.7 mm, 114 parts, among them J1 5055780871, J2 505578-0271, U1 IS31LT3360, U2 IS31LT3360, U3 IS31LT3360, U4 IS31LT3360, U5 IS31LT3360, U6 IS31LT3360

Commit message: added pca96...
Parts:
- removed R2: LDR03, OptoDevice:R_LDR_10x8.5mm_P7.6mm_Vertical
- removed R9: 100, Resistor_SMD:R_1206_3216Metric
- moved C2 39.6 mm to (70.0, 31.8)
- moved C3 39.6 mm to (77.4, 36.1)
- moved L1 39.6 mm to (66.9, 37.4)
- moved C1 39.6 mm to (71.8, 26.0)
- moved D1 39.6 mm to (66.2, 31.7)
- moved R1 39.6 mm to (73.8, 32.2)
- moved R8 39.6 mm to (74.5, 40.8)
- moved U1 39.6 mm to (73.8, 36.0)
- moved TH1 37.6 mm to (45.3, 75.9), turned to 180 degrees
- moved C13 36.6 mm to (74.7, 133.5)
- moved D12 36.6 mm to (190.5, 32.8)
- moved D20 36.6 mm to (128.3, 70.8)
- moved D30 36.6 mm to (157.1, 167.8)
- moved D45 36.6 mm to (68.4, 139.1)
- moved D51 36.6 mm to (160.1, 147.3)
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Connections:
- net Net-(J1-Pad5) renamed /NTC
- net Net-(J1-Pad7) renamed /12V_Fan
- J1 pad 8: Net-(J1-Pad8) -> /3.3V
- J2 pad 2: Net-(J1-Pad8) -> GND
- TH1 pad 2: GND -> /3.3V
Routing:
- net Net-(J1-Pad8): track 23.6 -> 0.00 mm
- net GND: track 524.8 -> 537.8 mm
- net Net-(D7-Pad1): track 0.00 -> 9.65 mm
- net Net-(D32-Pad1): track 0.00 -> 9.57 mm
- net Net-(D29-Pad1): track 0.00 -> 9.57 mm
- net Net-(D10-Pad1): track 0.00 -> 9.52 mm
- net Net-(D11-Pad1): track 0.00 -> 9.52 mm
- net Net-(D25-Pad1): track 0.00 -> 9.52 mm
- net Net-(D24-Pad1): track 0.00 -> 9.50 mm
- net Net-(D30-Pad1): track 0.00 -> 9.47 mm
- net Net-(D26-Pad1): track 0.00 -> 9.47 mm
- net Net-(D27-Pad1): track 0.00 -> 9.45 mm
- net Net-(D28-Pad1): track 0.00 -> 9.45 mm
- net Net-(D31-Pad1): track 0.00 -> 9.40 mm
- net Net-(D5-Pad1): track 0.00 -> 9.37 mm
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Other:
- board size 117.7 x 117.7 mm -> 186 x 170 mm
- net class Default: clearance 0.4 -> 0.2
- rule trace_clearance: 0.4 -> 0.2

Commit message: updates to Control board and LED light
Parts:
- moved C5 0.27 mm to (69.8, 57.1)
Routing:
- net Net-(D18-Pad1): track 19.0 -> 23.9 mm
- net GND: track 537.8 -> 541.5 mm
- net Net-(D17-Pad1): track 45.2 -> 48.2 mm
- net VCC: track 479.1 -> 476.6 mm
- net Net-(D6-Pad1): track 9.00 -> 9.70 mm

Commit message: minor changes
Parts:
- added REF**: MountingHole_3.2mm_M3_DIN965, MountingHole:MountingHole_3.2mm_M3_DIN965, F.Cu at (83.4, 152.8)
- added REF**: MountingHole_3.2mm_M3_DIN965, MountingHole:MountingHole_3.2mm_M3_DIN965, F.Cu at (188.5, 152.8)
- added REF**: MountingHole_3.2mm_M3_DIN965, MountingHole:MountingHole_3.2mm_M3_DIN965, F.Cu at (188.5, 47.8)
- added REF**: MountingHole_3.2mm_M3_DIN965, MountingHole:MountingHole_3.2mm_M3_DIN965, F.Cu at (83.5, 47.8)
Other:
- outline, holes or cut-outs redrawn
Changed lines of the file:
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@@
   (general
     (thickness 1.6)
-    (drawings 424)
+    (drawings 420)
     (tracks 708)
     (zones 0)
-    (modules 112)
+    (modules 116)
     (nets 86)
   )
@@
     (uvia_drill 0.1)
   )
+  (module MountingHole:MountingHole_3.2mm_M3_DIN965 (layer F.Cu)
+    (at 83.43 152.82)
+    (descr "Mounting Hole 3.2mm, no annular, M3, DIN965")
+    (tags "mounting hole 3.2mm no annular m3 din965")
+    (attr virtual)
+    (fp_text reference REF** (at 0 -3.8) (layer F.SilkS)
+      (effects (font (size 1 1) (thickness 0.15)))
+    )
+    (fp_text value MountingHole_3.2mm_M3_DIN965 (at 0 3.8) (layer F.Fab)
+      (effects (font (size 1 1) (thickness 0.15)))
+    )
+    (fp_text user %R (at 0.3 0) (layer F.Fab)
+      (effects (font (size 1 1) (thickness 0.15)))
+    )
+    (fp_circle (center 0 0) (end 2.8 0) (layer Cmts.User) (width 0.15))
+    (fp_circle (center 0 0) (end 3.05 0) (layer F.CrtYd) (width 0.05))
+    (pad 1 np_thru_hole circle (at 0 0) (size 3.2 3.2) (drill 3.2) (layers *.Cu *.Mask))
+  )
+  (module MountingHole:MountingHole_3.2mm_M3_DIN965 (layer F.Cu)
+    (at 188.49 152.84)
+    (descr "Mounting Hole 3.2mm, no annular, M3, DIN965")
+    (tags "mounting hole 3.2mm no annular m3 din965")
+    (attr virtual)
+    (fp_text reference REF** (at 0 -3.8) (layer F.SilkS)
+      (effects (font (size 1 1) (thickness 0.15)))
+    )
+    (fp_text value MountingHole_3.2mm_M3_DIN965 (at 0 3.8) (layer F.Fab)
+      (effects (font (size 1 1) (thickness 0.15)))
+    )
+    (fp_circle (center 0 0) (end 3.05 0) (layer F.CrtYd) (width 0.05))
+    (fp_circle (center 0 0) (end 2.8 0) (layer Cmts.User) (width 0.15))
+    (fp_text user %R (at 0.3 0) (layer F.Fab)
+      (effects (font (size 1 1) (thickness 0.15)))
+    )
+    (pad 1 np_thru_hole circle (at 0 0) (size 3.2 3.2) (drill 3.2) (layers *.Cu *.Mask))
+  )
+  (module MountingHole:MountingHole_3.2mm_M3_DIN965 (layer F.Cu)
+    (at 188.49 47.78)
+    (descr "Mounting Hole 3.2mm, no annular, M3, DIN965")
+    (tags "mounting hole 3.2mm no annular m3 din965")
+    (attr virtual)
+    (fp_text reference REF** (at 0 -3.8) (layer F.SilkS)
+      (effects (font (size 1 1) (thickness 0.15)))
+    )
+    (fp_text value MountingHole_3.2mm_M3_DIN965 (at 0 3.8) (layer F.Fab)
+      (effects (font (size 1 1) (thickness 0.15)))
+    )
+    (fp_text user %R (at 0.3 0) (layer F.Fab)
+      (effects (font (size 1 1) (thickness 0.15)))
+    )
+    (fp_circle (center 0 0) (end 2.8 0) (layer Cmts.User) (width 0.15))
+    (fp_circle (center 0 0) (end 3.05 0) (layer F.CrtYd) (width 0.05))
+    (pad 1 np_thru_hole circle (at 0 0) (size 3.2 3.2) (drill 3.2) (layers *.Cu *.Mask))
+  )
+  (module MountingHole:MountingHole_3.2mm_M3_DIN965 (layer F.Cu)
+    (at 83.45 47.83)
+    (descr "Mounting Hole 3.2mm, no annular, M3, DIN965")
+    (tags "mounting hole 3.2mm no annular m3 din965")
+    (attr virtual)
+    (fp_text reference REF** (at 0 -3.8) (layer F.SilkS)
+      (effects (font (size 1 1) (thickness 0.15)))
+    )
+    (fp_text value MountingHole_3.2mm_M3_DIN965 (at 0 3.8) (layer F.Fab)
+      (effects (font (size 1 1) (thickness 0.15)))
+    )
+    (fp_circle (center 0 0) (end 3.05 0) (layer F.CrtYd) (width 0.05))
+    (fp_circle (center 0 0) (end 2.8 0) (layer Cmts.User) (width 0.15))
+    (fp_text user %R (at 0.3 0) (layer F.Fab)
+      (effects (font (size 1 1) (thickness 0.15)))
+    )
+    (pad 1 np_thru_hole circle (at 0 0) (size 3.2 3.2) (drill 3.2) (layers *.Cu *.Mask))
+  )
   (module Kicad_mylib:JK3030AWT-00-0000-000A0UJ465E (layer F.Cu)
     (at 57.29 81.89 90)
@@
   (gr_line (start 158.42564 154.734141) (end 120.1637 115.929045) (layer Edge.Cuts) (width 0.2))
   (gr_line (start 115.312945 108.466692) (end 88.64573 135.326605) (layer Edge.Cuts) (width 0.2))
-  (gr_circle (center 188.46185 152.852022) (end 190.61185 152.852022) (layer Edge.Cuts) (width 0.2))
   (gr_arc (start 135.96185 100.352022) (end 100.987267 53.035902) (angle -75.97355982) (layer Edge.Cuts) (width 0.2))
   (gr_line (start 127.84718 79.703117) (end 100.987267 53.035902) (layer Edge.Cuts) (width 0.2))
   (gr_line (start 151.76 84.775) (end 156.610756 92.237353) (layer Edge.Cuts) (width 0.2))
   (gr_line (start 34.547079 14.609661) (end 220.547079 14.609661) (layer Edge.Cuts) (width 0.2))
-  (gr_circle (center 83.46185 152.852022) (end 85.61185 152.852022) (layer Edge.Cuts) (width 0.2))
   (gr_line (start 220.547079 14.609661) (end 220.547079 184.609661) (layer Edge.Cuts) (width 0.2))
   (gr_line (start 81.579731 122.815812) (end 120.384828 84.553873) (layer Edge.Cuts) (width 0.2))
@@
   (gr_arc (start 135.961648 100.352045) (end 183.277768 65.377462) (angle -75.97355982) (layer Edge.Cuts) (width 0.2))
   (gr_line (start 151.538873 116.150172) (end 144.07652 121.000928) (layer Edge.Cuts) (width 0.2))
-  (gr_circle (center 188.46185 47.852022) (end 190.61185 47.852022) (layer Edge.Cuts) (width 0.2))
   (gr_line (start 156.610756 92.237353) (end 183.277768 65.377462) (layer Edge.Cuts) (width 0.2))
   (gr_line (start 34.547079 184.609661) (end 34.547079 14.609661) (layer Edge.Cuts) (width 0.2))
   (gr_line (start 220.547079 184.609661) (end 34.547079 184.609661) (layer Edge.Cuts) (width 0.2))
-  (gr_circle (center 83.46185 47.852022) (end 85.61185 47.852022) (layer Edge.Cuts) (width 0.2))
   (gr_line (start 163.514825 95.082199) (end 163.514825 91.582199) (layer Dwgs.User) (width 0.2))
   (gr_line (start 175.821783 86.211602) (end 172.321783 86.211602) (layer Dwgs.User) (width 0.2))
