File: Projects/LED_DRIVER_with_fan_IS31LT3117/LED_Driver_ISSI_ALU_IS31LT3117.kicad_pcb (KiCad board)
At the start: 2 copper layers, 186 x 170 mm, 84 parts, among them IC1 IS31LT3117-ZLS4-TR, J1 43045-0809

Commit message: files after harddrive restore
Parts:
- removed H5: throughHole, MountingHole:MountingHole_6.4mm_M6
- C1: value 10u/EDK106M063A9GAA -> 10u 50V; footprint SamacSys_Parts:CAPAE660X565N -> Capacitor_SMD:CP_Elec_5x5.3
- moved D55 201.7 mm to (57.4, 155.3), turned to 90 degrees
- moved D38 197.2 mm to (168.2, 177.8), turned to 180 degrees
- moved D54 196.7 mm to (57.4, 143.2), turned to 90 degrees
- moved D36 194.3 mm to (145.9, 177.8), turned to 180 degrees
- moved D65 193.7 mm to (134.2, 173.8), turned to 180 degrees
- moved D34 192.1 mm to (123.8, 177.8), turned to 180 degrees
- moved H3 191.8 mm to (83.5, 152.9)
- moved D31 191.2 mm to (90.3, 177.8), turned to 180 degrees
- moved D33 190.0 mm to (112.6, 177.8), turned to 180 degrees
- moved D40 181.8 mm to (190.4, 177.8), turned to 180 degrees
- moved D32 180.2 mm to (101.5, 177.8), turned to 180 degrees
- moved D35 179.6 mm to (134.8, 177.8), turned to 180 degrees
- moved D25 177.1 mm to (213.8, 155.3), turned to 90 degrees
- moved D39 176.8 mm to (179.3, 177.8), turned to 180 degrees
- moved D37 171.0 mm to (157.1, 177.8), turned to 180 degrees
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Connections:
- J1 pad 1: /ADJ_LED -> GND
- J1 pad 2: GND -> /ADJ_LED
Routing:
- net /+48V: track 100.1 -> 600.6 mm
- net Net-(D25-Pad1): track 0.00 -> 126.3 mm
- net Net-(D45-Pad1): track 0.00 -> 102.3 mm
- net Net-(D60-Pad1): track 150.5 -> 76.4 mm
- net Net-(D10-Pad1): track 0.00 -> 69.4 mm
- net Net-(D40-Pad1): track 0.00 -> 56.1 mm
- net Net-(D55-Pad1): track 0.00 -> 50.4 mm
- net Net-(D15-Pad1): track 66.2 -> 111.6 mm
- net Net-(D30-Pad1): track 0.00 -> 32.3 mm
- net GND: track 82.1 -> 111.5 mm
- net Net-(D11-Pad1): track 0.00 -> 26.3 mm
- net Net-(D41-Pad1): track 0.00 -> 24.2 mm
- net Net-(D14-Pad1): track 0.00 -> 23.9 mm
- net Net-(D12-Pad1): track 0.00 -> 22.2 mm
- net Net-(D13-Pad1): track 0.00 -> 22.0 mm
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Other:
- board size 186 x 170 mm -> 170 x 170 mm
- net class Default: trace_width 0.45 -> 0.4
- net class power: trace_width 0.4 -> 0.8
