File: Projects/LED_DRIVER_with_fan_IS31LT3117/LED_Driver_ISSI_ALU_IS31LT3117.sch (KiCad schematic (older format))
At the start: 84 parts, among them IC1 IS31LT3117-ZLS4-TR, J1 43045-0809

Commit message: files after harddrive restore
Parts:
- removed C1: 10u/EDK106M063A9GAA, SamacSys_Parts:CAPAE660X565N, symbol SamacSys_Parts:EDK106M063A9GAA
- added C1: 10u 50V, Capacitor_SMD:CP_Elec_5x5.3, symbol Device:CP
- H5: footprint MountingHole:MountingHole_6.4mm_M6 -> MountingHole:MountingHole_8.4mm_M8
Other:
- note added: "Mates with: 43025-0800 and crimp terminals\n"
- note added: "Wurth part number:\n662008231722"
Changed lines of the file:
@@
 $EndComp
-Wire Wire Line
-	3000 6900 3000 7000
 Wire Wire Line
 	3600 7050 3600 6900
@@
 Wire Wire Line
 	3600 7650 3000 7650
-Wire Wire Line
-	3000 7650 3000 7500
 $Comp
 L power:GND #PWR02
@@
 Text Label 2300 4500 0    60   ~ 0
 48V_Fan
-Text Label 1500 4500 2    60   ~ 0
+Text Label 1500 4600 2    60   ~ 0
 ADJ_LED
 Text Label 1500 4700 2    60   ~ 0
@@
 	1    0    0    -1
 $EndComp
-Text Label 1500 4600 2    60   ~ 0
+Text Label 1500 4500 2    60   ~ 0
 GND
 Text Label 2300 4600 0    60   ~ 0
@@
 $EndComp
 Wire Wire Line
-	850  4650 850  4600
-Wire Wire Line
-	850  4600 1500 4600
-Wire Wire Line
 	1150 4800 1150 6900
 Wire Wire Line
@@
 Wire Wire Line
 	6700 5750 6700 5950
-$Comp
-L SamacSys_Parts:EDK106M063A9GAA C1
-U 1 1 5E32870A
-P 3000 7000
-F 0 "C1" H 3250 7267 50  0000 C CNN
-F 1 "10u/EDK106M063A9GAA" H 3250 7176 50  0000 C CNN
-F 2 "SamacSys_Parts:CAPAE660X565N" H 3350 7050 50  0001 L CNN
-F 3 "https://api.kemet.com/component-edge/download/specsheet/EDK106M063A9GAA.pdf" H 3350 6950 50  0001 L CNN
-F 4 "KEMET Aluminium Electrolytic Capacitor 10uF 63V dc 6.3mm Can - SMD, Radial EDK Series Aluminium Electrolytic" H 3350 6850 50  0001 L CNN "Description"
-F 5 "5.65" H 3350 6750 50  0001 L CNN "Height"
-F 6 "Kemet" H 3350 6650 50  0001 L CNN "Manufacturer_Name"
-F 7 "EDK106M063A9GAA" H 3350 6550 50  0001 L CNN "Manufacturer_Part_Number"
-F 8 "80-EDK106M063A9GAA" H 3350 6450 50  0001 L CNN "Mouser Part Number"
-F 9 "https://www.mouser.com/Search/Refine.aspx?Keyword=80-EDK106M063A9GAA" H 3350 6350 50  0001 L CNN "Mouser Price/Stock"
-F 10 "8707336" H 3350 6250 50  0001 L CNN "RS Part Number"
-F 11 "http://uk.rs-online.com/web/p/products/8707336" H 3350 6150 50  0001 L CNN "RS Price/Stock"
-F 12 "70097575" H 3350 6050 50  0001 L CNN "Allied_Number"
-F 13 "https://www.alliedelec.com/kemet-edk106m063a9gaa/70097575/" H 3350 5950 50  0001 L CNN "Allied Price/Stock"
-	1    3000 7000
-	0    1    1    0
-$EndComp
 Wire Wire Line
 	1150 4800 1500 4800
@@
 F 0 "H5" H 9100 8546 50  0000 L CNN
 F 1 "throughHole" H 9100 8455 50  0000 L CNN
-F 2 "MountingHole:MountingHole_6.4mm_M6" H 9000 8500 50  0001 C CNN
+F 2 "MountingHole:MountingHole_8.4mm_M8" H 9000 8500 50  0001 C CNN
 F 3 "~" H 9000 8500 50  0001 C CNN
 	1    9000 8500
 	1    0    0    -1
 $EndComp
+$Comp
+L Device:CP C1
+U 1 1 5E323314
+P 3000 7200
+F 0 "C1" H 3118 7246 50  0000 L CNN
+F 1 "10u 50V" H 3118 7155 50  0000 L CNN
+F 2 "Capacitor_SMD:CP_Elec_5x5.3" H 3038 7050 50  0001 C CNN
+F 3 "https://www.we-online.com/catalog/datasheet/865080642006.pdf" H 3000 7200 50  0001 C CNN
+	1    3000 7200
+	1    0    0    -1
+$EndComp
+Wire Wire Line
+	3000 6900 3000 7050
+Wire Wire Line
+	3000 7350 3000 7650
+Wire Wire Line
+	850  4500 850  4650
+Wire Wire Line
+	850  4500 1500 4500
+Text Notes 850  3700 0    60   ~ 0
+Mates with: 43025-0800 and crimp terminals\n
+Text Notes 1550 4100 0    60   ~ 0
+Wurth part number:\n662008231722
 $EndSCHEMATC

Commit message: added code
Parts:
- IC1: symbol SamacSys_Parts:IS31LT3117-ZLS4-TR -> LED_Driver_ISSI_ALU_IS31LT3117-rescue:IS31LT3117-ZLS4-TR-SamacSys_Parts
- J1: symbol SamacSys_Parts:43045-0809 -> LED_Driver_ISSI_ALU_IS31LT3117-rescue:43045-0809-SamacSys_Parts
Changed lines of the file:
@@
 EESchema Schematic File Version 4
-LIBS:LED_Driver_ISSI_ALU_IS31LT3117-cache
-EELAYER 29 0
+EELAYER 30 0
 EELAYER END
 $Descr A3 16535 11693
@@
 $EndComp
 $Comp
-L SamacSys_Parts:IS31LT3117-ZLS4-TR IC1
+L LED_Driver_ISSI_ALU_IS31LT3117-rescue:IS31LT3117-ZLS4-TR-SamacSys_Parts IC1
 U 1 1 5E591F90
 P 5100 6700
@@
 NTC
 $Comp
-L SamacSys_Parts:43045-0809 J1
+L LED_Driver_ISSI_ALU_IS31LT3117-rescue:43045-0809-SamacSys_Parts J1
 U 1 1 5E678007
 P 1500 4500

Commit message: updated PCB
Parts:
- C1: Manufacturer_Part_Number (none) -> 865080642006
- C3: Manufacturer_Part_Number (none) -> VE-330M1HTR-0607
Changed lines of the file:
@@
 F 2 "Resistor_SMD:R_0603_1608Metric" H 1900 5400 50  0001 C CNN
 F 3 "~" H 1900 5400 50  0001 C CNN
+F 4 "" H 1900 5350 50  0001 C CNN "Mouser Part Number"
 	1    1900 5350
 	0    1    1    0
@@
 F 2 "Capacitor_SMD:C_0805_2012Metric" H 3638 7050 50  0001 C CNN
 F 3 "~" H 3600 7200 50  0001 C CNN
+F 4 "" H 3600 7200 50  0001 C CNN "Manufacturer_Part_Number"
 	1    3600 7200
 	1    0    0    -1
@@
 F 2 "Capacitor_SMD:C_1206_3216Metric" H 6938 7550 50  0001 C CNN
 F 3 "~" H 6900 7700 50  0001 C CNN
+F 4 "" H 6900 7700 50  0001 C CNN "Manufacturer_Part_Number"
 	1    6900 7700
 	1    0    0    -1
@@
 F 2 "Capacitor_SMD:CP_Elec_6.3x7.7" H 6738 5450 50  0001 C CNN
 F 3 "https://www.mouser.com/Search/Refine.aspx?Keyword=140-VE330M1HTR0607" H 6700 5600 50  0001 C CNN
+F 4 "VE-330M1HTR-0607" H 6700 5600 50  0001 C CNN "Manufacturer_Part_Number"
 	1    6700 5600
 	1    0    0    -1
@@
 F 2 "Capacitor_SMD:CP_Elec_5x5.3" H 3038 7050 50  0001 C CNN
 F 3 "https://www.we-online.com/catalog/datasheet/865080642006.pdf" H 3000 7200 50  0001 C CNN
+F 4 "865080642006" H 3000 7200 50  0001 C CNN "Manufacturer_Part_Number"
 	1    3000 7200
 	1    0    0    -1
